File: carrier_board_v1/cm4-high-speed.kicad_sch (KiCad schematic)
At the start: 1 part

Commit message: -
Parts:
- added J3: USB4105-GF-A, USB4105-GF-A:GCT_USB4105-GF-A, symbol USB4105-GF-A:USB4105-GF-A
- added J3: 54548-2271, 54548-2271:MOLEX_54548-2271, symbol 54548-2271:54548-2271
- added R1, R4: 5.1k, Resistor_SMD:R_0603_1608Metric_Pad0.98x0.95mm_HandSolder, symbol Device:R
- added R5, R6: 2.2K 1%, Resistor_SMD:R_0402_1005Metric, symbol Device:R
- added R7, R8: 2.2K 1%, Resistor_SMD:R_0603_1608Metric_Pad0.98x0.95mm_HandSolder, symbol Device:R
- added U3: TPD2EUSB30, Package_TO_SOT_SMD:Texas_DRT-3, symbol Power_Protection:TPD2EUSB30
Connections:
- net GND: now also J3.1, J3.10, J3.13, J3.16, J3.19, J3.4, J3.7, J3.A1_B12 (GND), J3.B1_A12 (GND), R1.2, R4.2, R8.2, U3.3 (GND)
- net USB_OTG_ID: now reaches Module1.101 (USB_OTG_ID)
- net USB_OTG_ID: now also R7.2, R8.1
- net USB2_N: now reaches Module1.103 (USB2_N)
- net USB2_N: now also J3.A7 (DN1), J3.B7 (DN2), U3.2 (D-)
- net USB2_P: now reaches Module1.105 (USB2_P)
- net USB2_P: now also J3.A6 (DP1), J3.B6 (DP2), U3.1 (D+)
- net CAM0_D0_N: now reaches Module1.128 (CAM0_D0_N)
- net CAM0_D0_N: now also J3.2
- net CAM0_D0_P: now reaches Module1.130 (CAM0_D0_P)
- net CAM0_D0_P: now also J3.3
- net CAM0_D1_N: now reaches Module1.134 (CAM0_D1_N)
- net CAM0_D1_N: now also J3.5
- net CAM0_D1_P: now reaches Module1.136 (CAM0_D1_P)
- net CAM0_D1_P: now also J3.6
- net CAM0_C_N: now reaches Module1.140 (CAM0_C_N)
- net CAM0_C_N: now also J3.8
- net CAM0_C_P: now reaches Module1.142 (CAM0_C_P)
- net CAM0_C_P: now also J3.9
- new net: J3.B5 (CC2), R4.1
- new net: J3.A4_B9 (VBUS), J3.B4_A9 (VBUS), R7.1
- new net: J3.A5 (CC1), R1.1
- new net: J3.S1 (SHELL_GND), J3.S2 (SHELL_GND), J3.S3 (SHELL_GND), J3.S4 (SHELL_GND)
- new net: J3.SH1 (SHIELD), J3.SH2 (SHIELD)
- new net +3.3V: J3.22
- new net CAM_GPIO: J3.17
- new net GPIO_VREF: R5.1, R6.1
- new net SCL1: J3.20, J3.21, R5.2, R6.2
- no-connect marks 0 -> 59
Other:
- note added: "ESD protection"
- note added: "Raspberry Pi Camera Module connector"
- note added: "USB C for Infiray P2 Pro"
