File: prototype/cm4-high-speed.kicad_sch (KiCad schematic)
At the start: 1 part

Commit message: update
Parts:
- added J2: 54548-2271, 54548-2271:MOLEX_54548-2271, symbol 54548-2271:54548-2271
- added J3: USB4105-GF-A, USB4105-GF-A:GCT_USB4105-GF-A, symbol USB4105-GF-A:USB4105-GF-A
- added R1, R4: 5.1k, Resistor_SMD:R_0603_1608Metric_Pad0.98x0.95mm_HandSolder, symbol Device:R
- added R11, R12: 2.2K 1%, Resistor_SMD:R_0603_1608Metric_Pad0.98x0.95mm_HandSolder, symbol Device:R
- added R3, R5: 2.2K 1%, Resistor_SMD:R_0402_1005Metric, symbol Device:R
- added U2: TPD2EUSB30, Package_TO_SOT_SMD:Texas_DRT-3, symbol Power_Protection:TPD2EUSB30
Connections:
- net GND: now also J2.1, J2.10, J2.13, J2.16, J2.19, J2.4, J2.7, J3.A1_B12 (GND), J3.B1_A12 (GND), R1.2, R12.2, R4.2, U2.3 (GND)
- net USB_OTG_ID: now reaches Module1.101 (USB_OTG_ID)
- net USB_OTG_ID: now also R11.2, R12.1
- net USB2_N: now reaches Module1.103 (USB2_N)
- net USB2_N: now also J3.A7 (DN1), J3.B7 (DN2), U2.2 (D-)
- net USB2_P: now reaches Module1.105 (USB2_P)
- net USB2_P: now also J3.A6 (DP1), J3.B6 (DP2), U2.1 (D+)
- net CAM0_D0_N: now reaches Module1.128 (CAM0_D0_N)
- net CAM0_D0_N: now also J2.2
- net CAM0_D0_P: now reaches Module1.130 (CAM0_D0_P)
- net CAM0_D0_P: now also J2.3
- net CAM0_D1_N: now reaches Module1.134 (CAM0_D1_N)
- net CAM0_D1_N: now also J2.5
- net CAM0_D1_P: now reaches Module1.136 (CAM0_D1_P)
- net CAM0_D1_P: now also J2.6
- net CAM0_C_N: now reaches Module1.140 (CAM0_C_N)
- net CAM0_C_N: now also J2.8
- net CAM0_C_P: now reaches Module1.142 (CAM0_C_P)
- net CAM0_C_P: now also J2.9
- new net: J3.A5 (CC1), R1.1
- new net: J3.A4_B9 (VBUS), J3.B4_A9 (VBUS), R11.1
- new net: J3.B5 (CC2), R4.1
- new net: J3.S1 (SHELL_GND), J3.S2 (SHELL_GND), J3.S3 (SHELL_GND), J3.S4 (SHELL_GND)
- new net: J2.SH1 (SHIELD), J2.SH2 (SHIELD)
- new net +3.3V: J2.22
- new net CAM_GPIO: J2.17
- new net GPIO_VREF: R3.1, R5.1
- new net SCL1: J2.20, J2.21, R3.2, R5.2
- no-connect marks 0 -> 59
Other:
- note added: "ESD protection"
- note added: "Raspberry Pi Camera Module connector"
- note added: "USB C for Infiray P2 Pro"

Commit message: -
Connections:
- net CAM0_C_N is gone; now on net GND: J2.8, Module1.140 (CAM0_C_N)
- net CAM0_C_P is gone; now on net GND: J2.9, Module1.142 (CAM0_C_P)
- net CAM0_D0_N is gone; now on net GND: J2.2, Module1.128 (CAM0_D0_N)
- net CAM0_D1_N is gone; now on net GND: J2.5, Module1.134 (CAM0_D1_N)
- net USB2_P is gone; now on net USB2_N: J3.A6 (DP1), J3.B6 (DP2), Module1.105 (USB2_P), U2.1 (D+)
- net USB_OTG_ID is gone; now on net USB2_N: Module1.101 (USB_OTG_ID), R11.2, R12.1
