File: carrier_board_v1.kicad_pcb (KiCad board)
At the start: 2 copper layers, 40 x 55 mm, 33 parts, among them J1 B2B-PH-SM4-TB_LF__SN_, J3 54548-2271, J4 USB4105-GF-A, J6 USB4105-GF-A, J7 Conn_01x12_Pin, Q1 DMP3013SFV, U1 BQ25302RTER, U3 TPD2EUSB30, U5 TPS613222ADBZ

Commit message: -
Parts:
- removed C1: 22u, Capacitor_SMD:C_0201_0603Metric
- C2, C3, C4, C5, C6, C7, C8, CR1, D1, D2, J1, J3, J4, J6, L1, L2, Q1, R1, R10, R2, R3, R4, R6, R7, R8, R9, U1, U3, U5: moved to B.Cu
- moved R5 79.5 mm to (83.5, 127.6)
- moved D1 75.5 mm to (96.2, 126.5), turned to 90 degrees
- moved U3 63.5 mm to (154.6, 87.6), turned to 180 degrees
- moved C8 62.2 mm to (91.7, 119.8), turned to 180 degrees
- moved U5 61.8 mm to (88.4, 118.6), turned to 180 degrees
- moved D2 61.3 mm to (88.3, 112.5), turned to 180 degrees
- moved Q1 61.1 mm to (101.5, 124.8)
- moved C5 59.5 mm to (141.0, 127.2)
- moved L1 59.3 mm to (89.6, 121.4)
- moved C2 59.1 mm to (106.7, 117.1), turned to 90 degrees
- moved C3 55.7 mm to (141.5, 124.5)
- moved R1 51.9 mm to (141.1, 113.0)
- moved L2 51.3 mm to (137.8, 118.5), turned to 180 degrees
- moved R6 51.0 mm to (156.3, 124.9), turned to -90 degrees
- moved C4 50.8 mm to (136.9, 124.4), turned to 180 degrees
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Connections:
- C3 pad 1: /CM4 GPIO and power pins/VBUS -> +5V
- CR1 pad 1: /CM4 GPIO and power pins/VBUS -> +5V
- D1 pad 2: /CM4 GPIO and power pins/VBUS -> +5V
- J6 pad A4_B9: /CM4 GPIO and power pins/VBUS -> +5V
- J6 pad B4_A9: /CM4 GPIO and power pins/VBUS -> +5V
- U1 pad 16: /CM4 GPIO and power pins/VBUS -> +5V
Routing:
- net +5V: track 0.00 -> 37.3 mm
- net Net-(Q1-D): track 0.00 -> 20.3 mm, vias 0 -> 4
- net /CM4 GPIO and power pins/PMID: track 0.00 -> 9.20 mm, vias 0 -> 1
- net GND: track 0.00 -> 8.36 mm, vias 0 -> 6
- net Net-(U1-SW): track 0.00 -> 7.73 mm
- net /CM4 GPIO and power pins/GPIO10: track 0.00 -> 5.60 mm
- net /CM4 GPIO and power pins/REGN: track 0.00 -> 5.50 mm
- net /CM4 GPIO and power pins/GPIO11: track 0.00 -> 5.31 mm
- net /CM4 GPIO and power pins/GPIO9: track 0.00 -> 5.00 mm
- net Net-(J4-CC1): track 0.00 -> 2.98 mm
- net /CM4 Camera pins/USB2_P: track 0.00 -> 2.82 mm
- net /CM4 Camera pins/USB2_N: track 0.00 -> 2.82 mm
- net /CM4 Camera pins/VBUS: track 0.00 -> 2.77 mm
- net Net-(J4-CC2): track 0.00 -> 2.67 mm
- net Net-(U1-BTST): track 0.00 -> 2.23 mm
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- added copper zone on B.Cu, net GND
- added copper zone on F.Cu, net GND
Other:
- board size 40 x 55 mm -> 40.1 x 55.1 mm
- board text added: "RPi CM4 Carrier Board"
- board text removed: "RPi CM4 Carrier Template"
- board text removed: "Wireless Keepout"
- board text removed: "v01"

Commit message: what the fuck
Parts:
- added C1: 22u, Capacitor_SMD:C_0201_0603Metric, F.Cu at (117.4, 75.3)
- moved C8 94.7 mm to (183.2, 95.3)
- moved U5 94.7 mm to (179.9, 94.1)
- moved L1 94.7 mm to (181.1, 96.9)
- moved D2 87.7 mm to (174.2, 95.1), turned to -90 degrees
- moved J6 55.8 mm to (136.2, 78.9), turned to 0 degrees
- moved J4 54.6 mm to (137.2, 132.1), turned to 180 degrees
- moved D1 52.1 mm to (135.0, 91.9)
- moved Q1 51.2 mm to (141.9, 93.4), turned to 90 degrees
- moved U1 48.5 mm to (153.9, 82.4), turned to 0 degrees
- moved CR1 46.6 mm to (144.2, 81.9), turned to 90 degrees
- moved C5 45.1 mm to (150.3, 83.1), turned to 180 degrees
- moved R6 44.9 mm to (135.0, 85.4), turned to 90 degrees
- moved R4 42.8 mm to (135.1, 124.7), turned to 0 degrees
- moved C4 42.7 mm to (155.6, 86.0), turned to 90 degrees
- moved R8 42.7 mm to (146.7, 128.6), turned to 0 degrees
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Connections:
- J4 pad A4_B9: /CM4 Camera pins/VBUS -> +5V
- J4 pad B4_A9: /CM4 Camera pins/VBUS -> +5V
- R3 pad 1: /CM4 Camera pins/VBUS -> +5V
- R4 pad 1: /CM4 Camera pins/VBUS -> +5V
Routing:
- net /CM4 GPIO and power pins/PMID: track 9.20 -> 30.0 mm, vias 1 -> 0
- net +5V: track 37.3 -> 56.9 mm
- net /CM4 Camera pins/USB2_N: track 2.82 -> 18.8 mm, vias 0 -> 1
- net /CM4 Camera pins/USB2_P: track 2.82 -> 18.2 mm, vias 0 -> 1
- net Net-(Q1-D): track 20.3 -> 5.75 mm, vias 4 -> 1
- net Net-(D2-A): track 1.80 -> 8.63 mm
- net Net-(D1-K): track 0.00 -> 6.33 mm
- net /CM4 GPIO and power pins/GPIO10: track 5.60 -> 0.00 mm
- net /CM4 GPIO and power pins/REGN: track 5.50 -> 0.00 mm
- net Net-(U1-SW): track 7.73 -> 2.38 mm
- net /CM4 GPIO and power pins/GPIO11: track 5.31 -> 0.00 mm
- net /CM4 GPIO and power pins/GPIO9: track 5.00 -> 0.00 mm
- net /CM4 Camera pins/VBUS: track 2.77 -> 0.00 mm
- net Net-(U1-BTST): track 2.23 -> 3.17 mm
- net Net-(U1-ICHG_EN): track 0.90 -> 0.00 mm
- removed copper zone on B.Cu, net GND
- removed copper zone on F.Cu, net GND

Commit message: -
Parts:
- C1, R5: moved to B.Cu
- C6: moved to F.Cu
- moved R10 50.2 mm to (156.5, 102.5), turned to 180 degrees
- moved C1 49.1 mm to (160.4, 98.9), turned to -90 degrees
- moved C2 44.2 mm to (143.8, 93.0)
- moved C7 38.7 mm to (152.7, 106.5)
- moved C6 37.4 mm to (152.2, 89.0), turned to -90 degrees
- moved R2 37.3 mm to (147.5, 105.4), turned to 180 degrees
- moved L2 34.3 mm to (148.5, 98.0), turned to 0 degrees
- moved R5 28.9 mm to (135.3, 100.2), turned to 90 degrees
- moved C8 27.3 mm to (156.2, 99.1), turned to 90 degrees
- moved L1 26.5 mm to (154.6, 97.1), turned to -90 degrees
- moved U5 22.5 mm to (157.4, 95.8), turned to 90 degrees
- moved D2 18.5 mm to (156.4, 90.2), turned to 180 degrees
- moved R1 16.8 mm to (147.5, 104.2)
- moved J7 16.5 mm to (164.0, 117.2), turned to -90 degrees
- moved C4 15.2 mm to (145.8, 97.6), turned to -90 degrees
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Routing:
- net GND: track 7.98 -> 52.8 mm, vias 6 -> 17
- net Net-(Q1-D): track 5.75 -> 42.1 mm, vias 1 -> 3
- net /CM4 GPIO and power pins/TS: track 0.00 -> 19.8 mm, vias 0 -> 2
- net Net-(U1-ICHG_EN): track 0.00 -> 15.9 mm, vias 0 -> 2
- net +5V: track 56.9 -> 69.3 mm, vias 0 -> 3
- net /CM4 GPIO and power pins/PMID: track 30.0 -> 35.6 mm
- net Net-(U1-SW): track 2.38 -> 7.05 mm
- net /CM4 GPIO and power pins/REGN: track 0.00 -> 4.37 mm, vias 0 -> 1
- net Net-(D1-K): track 6.33 -> 9.02 mm
- net (no net): track 0.00 -> 1.75 mm
- net Net-(U1-BTST): track 3.17 -> 4.34 mm

Commit message: almost ready
Parts:
- C6: moved to B.Cu
- moved J7 27.9 mm to (136.1, 117.2), turned to 90 degrees
- moved D2 24.3 mm to (143.6, 110.8), turned to 90 degrees
- moved R2 20.7 mm to (158.5, 87.9), turned to 90 degrees
- moved C1 20.7 mm to (146.9, 114.5), turned to 180 degrees
- moved C7 20.1 mm to (163.3, 89.5)
- moved R10 18.5 mm to (142.9, 90.0), turned to 0 degrees
- moved CR1 18.2 mm to (129.9, 89.6), turned to 180 degrees
- moved R1 17.0 mm to (158.6, 91.3), turned to 90 degrees
- moved U5 16.2 mm to (148.1, 109.1), turned to 0 degrees
- moved C8 11.6 mm to (145.3, 103.2), turned to 180 degrees
- moved Q1 11.6 mm to (151.3, 100.5), turned to 0 degrees
- moved L1 10.9 mm to (147.1, 105.0), turned to 90 degrees
- moved C2 6.47 mm to (145.1, 99.3), turned to -90 degrees
- moved C3 6.18 mm to (143.2, 96.4), turned to 180 degrees
- moved R5 5.90 mm to (141.2, 101.3)
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Connections:
- U1 pad V: (no net) -> GND
Routing:
- net GND: track 52.8 -> 0.00 mm, vias 17 -> 0
- net /CM4 GPIO and power pins/REGN: track 4.37 -> 18.8 mm, vias 1 -> 2
- net Net-(U1-ICHG_EN): track 15.9 -> 2.90 mm, vias 2 -> 0
- net /CM4 GPIO and power pins/PMID: track 35.6 -> 26.1 mm
- net Net-(Q1-D): track 42.1 -> 32.9 mm, vias 3 -> 0
- net +5V: track 69.3 -> 75.0 mm, vias 3 -> 0
- net Net-(D1-K): track 9.02 -> 13.1 mm, vias 0 -> 2
- net /CM4 GPIO and power pins/TS: track 19.8 -> 16.1 mm
- net Net-(U1-BTST): track 4.34 -> 5.40 mm
- net Net-(J6-CC2): track 1.42 -> 2.30 mm
- net Net-(U1-SW): track 7.05 -> 6.39 mm
- net Net-(D2-A): track 8.63 -> 8.04 mm
- added copper zone on B.Cu, net GND
- added copper zone on F.Cu, net GND

Commit message: -
Connections:
- J3 pad 22: +3.3v -> +3.3V
- U1 pad V: GND -> (no net)
Routing:
- net /CM4 GPIO and power pins/GPIO14: track 0.00 -> 65.0 mm
- net +3.3V: track 0.00 -> 53.1 mm, vias 0 -> 1
- net /CM4 GPIO and power pins/GPIO3: track 0.00 -> 50.9 mm, vias 0 -> 2
- net +5V: track 75.0 -> 122.1 mm, vias 0 -> 3
- net /CM4 GPIO and power pins/GPIO2: track 0.00 -> 42.2 mm
- net CAM_GPIO: track 0.00 -> 38.7 mm, vias 0 -> 3
- net /CM4 GPIO and power pins/GPIO15: track 0.00 -> 31.7 mm, vias 0 -> 2
- net SCL0: track 0.00 -> 30.2 mm, vias 0 -> 1
- net SDA0: track 0.00 -> 30.0 mm, vias 0 -> 1
- net /CM4 GPIO and power pins/nRPIBOOT: track 0.00 -> 27.5 mm
- net /CM4 GPIO and power pins/GPIO10: track 0.00 -> 21.0 mm
- net /CM4 GPIO and power pins/GPIO8: track 0.00 -> 19.6 mm
- net /CM4 GPIO and power pins/GPIO9: track 0.00 -> 17.9 mm
- net /CM4 GPIO and power pins/GPIO7: track 0.00 -> 17.1 mm
- net /CM4 GPIO and power pins/GPIO11: track 0.00 -> 15.9 mm
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
Commit message: -
Parts:
- removed R7, R8: 2.2K 1%, Resistor_SMD:R_0201_0603Metric
- moved C3 2.32 mm to (141.0, 95.6)
- moved U3 1.08 mm to (137.9, 124.7)
- moved CR1 0.30 mm to (130.2, 89.6)
- renumbered Module1 to V1
Connections:
- V1 pad 88: +1.8V -> unconnected-(Module1A-+1.8v_(Output)-Pad88)
- V1 pad 90: +1.8V -> unconnected-(Module1A-+1.8v_(Output)-Pad90)
Routing:
- net unconnected-(J3-SHIELD-PadSH1): track 0.00 -> 17.5 mm
- net Net-(J4-SHELL_GND-PadS1): track 0.00 -> 17.0 mm
- net +5V: track 122.1 -> 136.3 mm, vias 3 -> 6
- net +3.3V: track 53.1 -> 63.2 mm, vias 1 -> 3
- net GND: track 0.00 -> 6.43 mm, vias 0 -> 102
- net /CM4 Camera pins/USB2_P: track 18.7 -> 23.4 mm
- net /CM4 Camera pins/CAM0_D1_N: track 0.00 -> 4.58 mm, vias 0 -> 1
- net /CM4 Camera pins/USB2_N: track 19.1 -> 22.8 mm
- net (no net): track 1.75 -> 0.00 mm
- net /CM4 GPIO and power pins/GPIO14: track 65.0 -> 66.1 mm
- net /CM4 Camera pins/CAM0_D0_N: track 4.46 -> 5.18 mm
Other:
- board text added: "3v3"
- board text added: "B"
- board text added: "CM4 Carrier Board"
- board text added: "GND"
- board text added: "P10"
- board text added: "P11"
- board text added: "P14"
- board text added: "P15"
- board text added: "P2"
- board text added: "P3"
- board text added: "P7"
- board text added: "P8"
- board text added: "P9"
- board text removed: "RPi CM4 Carrier Board"
