File: carrier_board_v1.kicad_pcb (KiCad board)
At the start: 2 copper layers, 40.1 x 55.1 mm, 31 parts, among them J1 B2B-PH-SM4-TB_LF__SN_, J3 54548-2271, J4 USB4105-GF-A, J6 USB4105-GF-A, J7 Conn_01x12_Pin, Q1 DMP3013SFV, U1 BQ25302RTER, U3 TPD2EUSB30, U5 TPS613222ADBZ

Commit message: -
Parts:
- moved R1 1.85 mm to (160.2, 92.2)
- moved R4 0.25 mm to (136.2, 124.5)
Routing:
- net /CM4 GPIO and power pins/REGN: track 18.8 -> 20.5 mm
- net /CM4 GPIO and power pins/TS: track 16.1 -> 17.8 mm
- net GND: vias 102 -> 101
Changed lines of the file:
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@@
   )
   (footprint "Resistor_SMD:R_1206_3216Metric" (layer "B.Cu")
-    (at 158.55 91.305 90)
+    (at 160.15 92.2375 90)
     (descr "Resistor SMD 1206 (3216 Metric), square (rectangular) end terminal, IPC_7351 nominal, (Body size source: IPC-SM-782 page 72, https://www.pcb-3d.com/wordpress/wp-content/uploads/ipc-sm-782a_amendment_1_and_2.pdf), generated with kicad-footprint-generator")
     (tags "resistor")
@@
   )
   (footprint "Resistor_SMD:R_0402_1005Metric" (layer "B.Cu")
-    (at 136.48 124.625)
+    (at 136.24 124.55)
     (descr "Resistor SMD 0402 (1005 Metric), square (rectangular) end terminal, IPC_7351 nominal, (Body size source: IPC-SM-782 page 72, https://www.pcb-3d.com/wordpress/wp-content/uploads/ipc-sm-782a_amendment_1_and_2.pdf), generated with kicad-footprint-generator")
     (tags "resistor")
@@
     (property "ki_keywords" "R res resistor")
     (attr smd)
-    (fp_text reference "R4" (at 0 1.17 180) (layer "B.SilkS")
+    (fp_text reference "R4" (at -2.24 0.3 180) (layer "B.SilkS")
         (effects (font (size 1 1) (thickness 0.15)) (justify mirror))
     )
@@
   )
   (segment (start 164.175 97.3) (end 163.85 97.625) (width 0.2) (layer "F.Cu") (net 1))
-  (segment (start 134.389085 112.335911) (end 141.62501 105.099986) (width 1.36703) (layer "F.Cu") (net 1))
   (segment (start 151.15 105.1) (end 141.625024 105.1) (width 1.36703) (layer "F.Cu") (net 1))
   (segment (start 165 98.1) (end 164.325 98.1) (width 0.2) (layer "F.Cu") (net 1))
+  (segment (start 141.62501 105.099986) (end 134.389085 112.335911) (width 1.36703) (layer "F.Cu") (net 1))
   (segment (start 165 96.5) (end 163.875 96.5) (width 0.2) (layer "F.Cu") (net 1))
   (segment (start 163.85 96.975) (end 163.85 96.475) (width 0.2) (layer "F.Cu") (net 1))
@@
   (segment (start 164.225 96.1) (end 163.85 96.475) (width 0.2) (layer "F.Cu") (net 1))
   (segment (start 165 96.1) (end 164.225 96.1) (width 0.2) (layer "F.Cu") (net 1))
-  (segment (start 134.389085 122.844585) (end 134.389085 112.335911) (width 1.36703) (layer "F.Cu") (net 1))
   (segment (start 164.325 98.1) (end 163.85 97.625) (width 0.2) (layer "F.Cu") (net 1))
   (segment (start 141.625024 105.1) (end 141.62501 105.099986) (width 1.36703) (layer "F.Cu") (net 1))
+  (segment (start 134.389085 112.335911) (end 134.389085 122.844585) (width 1.36703) (layer "F.Cu") (net 1))
   (segment (start 163.925 97.7) (end 163.85 97.625) (width 0.2) (layer "F.Cu") (net 1))
   (segment (start 165.000053 96.500053) (end 165 96.5) (width 0.2) (layer "F.Cu") (net 1))
   (segment (start 165 97.7) (end 163.925 97.7) (width 0.2) (layer "F.Cu") (net 1))
   (segment (start 163.925 96.9) (end 163.85 96.975) (width 0.2) (layer "F.Cu") (net 1))
-  (segment (start 134.389085 122.844585) (end 135.33475 123.79025) (width 1.36703) (layer "F.Cu") (net 1))
   (segment (start 163.85 97.625) (end 163.85 96.975) (width 0.2) (layer "F.Cu") (net 1))
   (segment (start 165 96.9) (end 163.925 96.9) (width 0.2) (layer "F.Cu") (net 1))
@@
   (via (at 141.62501 105.099986) (size 0.6) (drill 0.3) (layers "F.Cu" "B.Cu") (net 1))
   (via (at 151.15 105.1) (size 0.6) (drill 0.3) (layers "F.Cu" "B.Cu") (net 1))
-  (via (at 135.33475 123.79025) (size 0.59) (drill 0.3) (layers "F.Cu" "B.Cu") (net 1))
+  (via (at 134.389085 122.844585) (size 0.59) (drill 0.3) (layers "F.Cu" "B.Cu") (net 1))
+  (segment (start 135.73 124.55) (end 135.5195 124.55) (width 0.1524) (layer "B.Cu") (net 1))
   (segment (start 144.4875 96.4625) (end 143.19443 97.75557) (width 1.36703) (layer "B.Cu") (net 1))
   (segment (start 139.4125 91.2625) (end 142.6625 94.5125) (width 1.36703) (layer "B.Cu") (net 1))
@@
   (segment (start 146.625 91) (end 146.625 92.375) (width 0.2) (layer "B.Cu") (net 1))
   (segment (start 135.4 89.65) (end 137.8 89.65) (width 1.36703) (layer "B.Cu") (net 1))
-  (segment (start 136.0951 127.2455) (end 136.0951 124.5506) (width 0.6) (layer "B.Cu") (net 1))
   (segment (start 142.4125 94.5125) (end 142.6625 94.5125) (width 0.2) (layer "B.Cu") (net 1))
   (segment (start 143.6 112.875) (end 147.4 112.875) (width 1.36703) (layer "B.Cu") (net 1))
@@
   (segment (start 140.8948 127.2718) (end 140.8948 126.044439) (width 0.6) (layer "B.Cu") (net 1))
   (segment (start 156.525 108.25) (end 153.375 105.1) (width 1.36703) (layer "B.Cu") (net 1))
-  (segment (start 136.0942 127.2464) (end 136.0951 127.2455) (width 0.6) (layer "B.Cu") (net 1))
   (segment (start 132.05 89.65) (end 135.4 89.65) (width 1.36703) (layer "B.Cu") (net 1))
-  (segment (start 136.0951 124.5506) (end 135.33475 123.79025) (width 0.6) (layer "B.Cu") (net 1))
   (segment (start 141.55 95.625) (end 142.6625 94.5125) (width 0.2) (layer "B.Cu") (net 1))
+  (segment (start 135.5195 124.55) (end 135.33475 124.73475) (width 0.1524) (layer "B.Cu") (net 1))
   (segment (start 163.45 101.325) (end 163.45 97.85) (width 1.36703) (layer "B.Cu") (net 1))
   (segment (start 138.225 92.45) (end 139.4125 91.2625) (width 1.36703) (layer "B.Cu") (net 1))
@@
   (segment (start 140.71025 123.66025) (end 140.28975 123.66025) (width 0.6) (layer "B.Cu") (net 1))
   (segment (start 147.2 113.075) (end 147.4 112.875) (width 0.4) (layer "B.Cu") (net 1))
+  (segment (start 135.33475 123.79025) (end 134.389085 122.844585) (width 0.6) (layer "B.Cu") (net 1))
   (segment (start 146.625 92.375) (end 145.725 93.275) (width 0.2) (layer "B.Cu") (net 1))
   (segment (start 163.450053 96.500053) (end 163.45 96.5) (width 0.4) (layer "B.Cu") (net 1))
@@
   (segment (start 138.225 95.65) (end 138.225 92.45) (width 1.36703) (layer "B.Cu") (net 1))
   (segment (start 141.2649 125.674339) (end 141.2649 124.2149) (width 0.6) (layer "B.Cu") (net 1))
+  (segment (start 135.33475 124.73475) (end 135.33475 123.79025) (width 0.6) (layer "B.Cu") (net 1))
   (segment (start 163.45 97.2) (end 163.45 97.85) (width 1.36703) (layer "B.Cu") (net 1))
   (segment (start 163.45 96.5) (end 163.45 97.2) (width 1.36703) (layer "B.Cu") (net 1))
+  (segment (start 136.0942 125.4942) (end 135.33475 124.73475) (width 0.6) (layer "B.Cu") (net 1))
+  (segment (start 136.0942 127.2464) (end 136.0942 125.4942) (width 0.6) (layer "B.Cu") (net 1))
   (via (at 165.15 124.35) (size 0.6) (drill 0.3) (layers "F.Cu" "B.Cu") (free) (net 2))
   (via (at 137.375 105.675) (size 0.6) (drill 0.3) (layers "F.Cu" "B.Cu") (free) (net 2))
@@
   (via (at 150.85 103.275) (size 0.6) (drill 0.3) (layers "F.Cu" "B.Cu") (free) (net 2))
   (via (at 154.675 114.5) (size 0.6) (drill 0.3) (layers "F.Cu" "B.Cu") (free) (net 2))
-  (via (at 160.85 94.1) (size 0.6) (drill 0.3) (layers "F.Cu" "B.Cu") (free) (net 2))
   (via (at 132.75 92.7) (size 0.6) (drill 0.3) (layers "F.Cu" "B.Cu") (free) (net 2))
   (via (at 134.225 102.975) (size 0.6) (drill 0.3) (layers "F.Cu" "B.Cu") (free) (net 2))
@@
   (segment (start 150.6728 95.5548) (end 149.9454 94.8274) (width 0.2) (layer "B.Cu") (net 5))
   (segment (start 145.525 92.525) (end 144.95 91.95) (width 0.4) (layer "F.Cu") (net 6))
-  (segment (start 158.575 92.525) (end 145.525 92.525) (width 0.4) (layer "F.Cu") (net 6))
-  (via (at 158.575 92.525) (size 0.6) (drill 0.3) (layers "F.Cu" "B.Cu") (net 6))
+  (segment (start 158.575 94.4) (end 156.7 92.525) (width 0.4) (layer "F.Cu") (net 6))
+  (segment (start 156.7 92.525) (end 145.525 92.525) (width 0.4) (layer "F.Cu") (net 6))
+  (via (at 158.575 94.4) (size 0.6) (drill 0.3) (layers "F.Cu" "B.Cu") (net 6))
   (via (at 144.95 91.95) (size 0.6) (drill 0.3) (layers "F.Cu" "B.Cu") (net 6))
   (segment (start 145.25 90.45) (end 145.975 90.45) (width 0.2) (layer "B.Cu") (net 6))
@@
   (segment (start 144.95 91.95) (end 144.95 91.55) (width 0.4) (layer "B.Cu") (net 6))
   (segment (start 144.55 91.15) (end 143.25 91.15) (width 0.2) (layer "B.Cu") (net 6))
-  (segment (start 158.575 91.625) (end 158.575 92.525) (width 0.4) (layer "B.Cu") (net 6))
   (segment (start 144.95 91.55) (end 144.55 91.15) (width 0.4) (layer "B.Cu") (net 6))
   (segment (start 145.975 90.45) (end 146 90.475) (width 0.2) (layer "B.Cu") (net 6))
+  (segment (start 159.275 93.7) (end 158.575 94.4) (width 0.1524) (layer "B.Cu") (net 6))
+  (segment (start 160.15 93.7) (end 159.275 93.7) (width 0.1524) (layer "B.Cu") (net 6))
   (segment (start 152.575 91.15) (end 152.525 91.1) (width 0.2) (layer "B.Cu") (net 7))
   (segment (start 152.525 91.1332) (end 152.525 91.1) (width 1) (layer "B.Cu") (net 7))
@@
   (segment (start 148.8 89.475) (end 150.575 89.475) (width 0.2) (layer "B.Cu") (net 8))
   (segment (start 158.55 90.95) (end 158.55 89.525) (width 0.4) (layer "B.Cu") (net 8))
+  (segment (start 158.725 90.775) (end 158.55 90.95) (width 0.1524) (layer "B.Cu") (net 8))
   (segment (start 158.55 89.425) (end 158.6 89.475) (width 0.4) (layer "B.Cu") (net 8))
   (segment (start 158.55 88.175) (end 158.55 89.425) (width 0.4) (layer "B.Cu") (net 8))
+  (segment (start 160.15 90.775) (end 158.725 90.775) (width 0.1524) (layer "B.Cu") (net 8))
   (segment (start 148.55 99.55) (end 141.675 99.55) (width 1.36703) (layer "F.Cu") (net 9))
   (via (at 141.675 99.55) (size 0.6) (drill 0.3) (layers "F.Cu" "B.Cu") (net 9))

Commit message: _
Parts:
- moved C2 0.17 mm to (145.2, 99.4)
- moved R3 0.12 mm to (140.8, 124.7)
Routing:
- net +5V: track 136.8 -> 138.9 mm, vias 6 -> 7
Changed lines of the file:
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@@
   )
   (footprint "Package_TO_SOT_SMD:Texas_DRT-3" (layer "B.Cu")
-    (at 137.95 124.725)
+    (at 137.95 124.675)
     (descr "Texas Instrument DRT-3 1x0.8mm Pitch 0.7mm http://www.ti.com/lit/ds/symlink/tpd2eusb30.pdf")
     (tags "DRT-3 1x0.8mm Pitch 0.7mm")
@@
   )
   (footprint "Resistor_SMD:R_0402_1005Metric" (layer "B.Cu")
-    (at 140.87 124.6 180)
+    (at 140.76 124.65 180)
     (descr "Resistor SMD 0402 (1005 Metric), square (rectangular) end terminal, IPC_7351 nominal, (Body size source: IPC-SM-782 page 72, https://www.pcb-3d.com/wordpress/wp-content/uploads/ipc-sm-782a_amendment_1_and_2.pdf), generated with kicad-footprint-generator")
     (tags "resistor")
@@
     (property "ki_keywords" "R res resistor")
     (attr smd)
-    (fp_text reference "R3" (at 0 1.17) (layer "B.SilkS")
+    (fp_text reference "R3" (at -2.04 -0.05) (layer "B.SilkS")
         (effects (font (size 1 1) (thickness 0.15)) (justify mirror))
     )
@@
   )
   (footprint "Capacitor_SMD:C_0603_1608Metric" (layer "B.Cu")
-    (at 144.8692 101.7778 180)
+    (at 144.825 101.8 180)
     (descr "Capacitor SMD 0603 (1608 Metric), square (rectangular) end terminal, IPC_7351 nominal, (Body size source: IPC-SM-782 page 76, https://www.pcb-3d.com/wordpress/wp-content/uploads/ipc-sm-782a_amendment_1_and_2.pdf), generated with kicad-footprint-generator")
     (tags "capacitor")
@@
   )
   (footprint "Capacitor_SMD:C_0805_2012Metric" (layer "B.Cu")
-    (at 145.05 99.32 -90)
+    (at 145.2 99.4 -90)
     (descr "Capacitor SMD 0805 (2012 Metric), square (rectangular) end terminal, IPC_7351 nominal, (Body size source: IPC-SM-782 page 76, https://www.pcb-3d.com/wordpress/wp-content/uploads/ipc-sm-782a_amendment_1_and_2.pdf, https://docs.google.com/spreadsheets/d/1BsfQQcO9C6DZCsRaXUlFlo91Tg2WpOkGARC1WS5S8t0/edit?usp=sharing), generated with kicad-footprint-generator")
     (tags "capacitor")
@@
     (property "ki_keywords" "cap capacitor")
     (attr smd)
-    (fp_text reference "C2" (at -1.1236 1.7432 -180) (layer "B.SilkS")
+    (fp_text reference "C2" (at -0.95 2.05 -180) (layer "B.SilkS")
         (effects (font (size 1 1) (thickness 0.15)) (justify mirror))
     )
@@
     (property "ki_keywords" "R res resistor")
     (attr smd)
-    (fp_text reference "R4" (at -2.24 0.3 180) (layer "B.SilkS")
+    (fp_text reference "R4" (at -2.59 0.3 180) (layer "B.SilkS")
         (effects (font (size 1 1) (thickness 0.15)) (justify mirror))
     )
@@
   )
   (segment (start 164.175 97.3) (end 163.85 97.625) (width 0.2) (layer "F.Cu") (net 1))
+  (segment (start 163.249998 97.099998) (end 163.249998 96.900002) (width 0.2) (layer "F.Cu") (net 1))
   (segment (start 151.15 105.1) (end 141.625024 105.1) (width 1.36703) (layer "F.Cu") (net 1))
   (segment (start 165 98.1) (end 164.325 98.1) (width 0.2) (layer "F.Cu") (net 1))
+  (segment (start 163.45 97.3) (end 163.249998 97.099998) (width 0.2) (layer "F.Cu") (net 1))
   (segment (start 141.62501 105.099986) (end 134.389085 112.335911) (width 1.36703) (layer "F.Cu") (net 1))
   (segment (start 165 96.5) (end 163.875 96.5) (width 0.2) (layer "F.Cu") (net 1))
+  (segment (start 163.25 96.9) (end 164.2 96.9) (width 0.2) (layer "F.Cu") (net 1))
   (segment (start 163.85 96.975) (end 163.85 96.475) (width 0.2) (layer "F.Cu") (net 1))
   (segment (start 165 97.3) (end 164.175 97.3) (width 0.2) (layer "F.Cu") (net 1))
+  (segment (start 163.249998 96.900002) (end 163.25 96.9) (width 0.2) (layer "F.Cu") (net 1))
   (segment (start 164.225 96.1) (end 163.85 96.475) (width 0.2) (layer "F.Cu") (net 1))
   (segment (start 165 96.1) (end 164.225 96.1) (width 0.2) (layer "F.Cu") (net 1))
+  (segment (start 165 96.9) (end 164.2 96.9) (width 0.2) (layer "F.Cu") (net 1))
   (segment (start 164.325 98.1) (end 163.85 97.625) (width 0.2) (layer "F.Cu") (net 1))
   (segment (start 141.625024 105.1) (end 141.62501 105.099986) (width 1.36703) (layer "F.Cu") (net 1))
@@
   (segment (start 165.000053 96.500053) (end 165 96.5) (width 0.2) (layer "F.Cu") (net 1))
   (segment (start 165 97.7) (end 163.925 97.7) (width 0.2) (layer "F.Cu") (net 1))
+  (segment (start 164.175 97.3) (end 163.45 97.3) (width 0.2) (layer "F.Cu") (net 1))
   (segment (start 163.925 96.9) (end 163.85 96.975) (width 0.2) (layer "F.Cu") (net 1))
   (segment (start 163.85 97.625) (end 163.85 96.975) (width 0.2) (layer "F.Cu") (net 1))
-  (segment (start 165 96.9) (end 163.925 96.9) (width 0.2) (layer "F.Cu") (net 1))
+  (segment (start 164.2 96.9) (end 163.925 96.9) (width 0.2) (layer "F.Cu") (net 1))
   (segment (start 163.875 96.5) (end 163.85 96.475) (width 0.2) (layer "F.Cu") (net 1))
   (via (at 163.85 96.475) (size 0.6) (drill 0.3) (layers "F.Cu" "B.Cu") (net 1))
@@
   (via (at 151.15 105.1) (size 0.6) (drill 0.3) (layers "F.Cu" "B.Cu") (net 1))
   (via (at 134.389085 122.844585) (size 0.59) (drill 0.3) (layers "F.Cu" "B.Cu") (net 1))
+  (via (at 163.15 97) (size 0.6) (drill 0.3) (layers "F.Cu" "B.Cu") (net 1))
   (segment (start 135.73 124.55) (end 135.5195 124.55) (width 0.1524) (layer "B.Cu") (net 1))
   (segment (start 144.4875 96.4625) (end 143.19443 97.75557) (width 1.36703) (layer "B.Cu") (net 1))
@@
   (segment (start 147.125 100.86) (end 147.125 101.625) (width 1.36703) (layer "B.Cu") (net 3))
   (segment (start 147.225 100.21) (end 147.125 100.11) (width 0.4) (layer "B.Cu") (net 3))
-  (segment (start 145.05 98.975) (end 145.625 98.975) (width 0.4) (layer "B.Cu") (net 3))
-  (segment (start 145.625 98.975) (end 147.125 97.475) (width 0.4) (layer "B.Cu") (net 3))
+  (segment (start 145.05 98.37) (end 146.23 98.37) (width 0.4) (layer "B.Cu") (net 3))
+  (segment (start 146.23 98.37) (end 147.125 97.475) (width 0.4) (layer "B.Cu") (net 3))
   (segment (start 147.125 101.625) (end 147.125 102.938) (width 0.4) (layer "B.Cu") (net 3))
   (segment (start 147.24 101.51) (end 147.125 101.625) (width 0.4) (layer "B.Cu") (net 3))
@@
   (segment (start 130.2 112.5) (end 130 112.3) (width 0.2) (layer "F.Cu") (net 30))
   (via (at 130 112.3) (size 0.508) (drill 0.254) (layers "F.Cu" "B.Cu") (net 30))
+  (segment (start 137.5 124.55) (end 137.5 124.25) (width 0.2) (layer "B.Cu") (net 30))
   (segment (start 137.7375 127.05) (end 137.7375 127.825) (width 0.2) (layer "B.Cu") (net 30))
   (segment (start 137.3 124.75) (end 137.5 124.55) (width 0.2) (layer "B.Cu") (net 30))
@@
   (segment (start 138.0125 128.1) (end 138.4 128.1) (width 0.2) (layer "B.Cu") (net 30))
   (segment (start 137.7375 126.3875) (end 137.3 125.95) (width 0.2) (layer "B.Cu") (net 30))
+  (segment (start 137.5 124.25) (end 137.5 124.0682) (width 0.2) (layer "B.Cu") (net 30))
   (segment (start 129.206801 112.474999) (end 129.825001 112.474999) (width 0.2) (layer "B.Cu") (net 30))
   (segment (start 137.3 125.95) (end 137.3 124.75) (width 0.2) (layer "B.Cu") (net 30))
-  (segment (start 137.5 124.55) (end 137.5 124.0682) (width 0.2) (layer "B.Cu") (net 30))
+  (segment (start 137.6 124.25) (end 137.5 124.25) (width 0.2) (layer "B.Cu") (net 30))
   (segment (start 137.7375 127.825) (end 138.0125 128.1) (width 0.2) (layer "B.Cu") (net 30))
   (segment (start 138.7375 127.7625) (end 138.7375 127.05) (width 0.2) (layer "B.Cu") (net 30))
@@
   (segment (start 136.7292 127.2718) (end 136.7292 124.6048) (width 0.25) (layer "B.Cu") (net 32))
   (segment (start 139.7264 127.2718) (end 139.7264 126.2236) (width 0.25) (layer "B.Cu") (net 33))
-  (segment (start 140.5646 125.3854) (end 140.5646 124.5794) (width 0.25) (layer "B.Cu") (net 33))
-  (segment (start 139.7264 126.2236) (end 140.5646 125.3854) (width 0.25) (layer "B.Cu") (net 33))
+  (segment (start 140.3 125.65) (end 140.3 124.66) (width 0.25) (layer "B.Cu") (net 33))
+  (segment (start 140.3 124.66) (end 140.36 124.6) (width 0.25) (layer "B.Cu") (net 33))
+  (segment (start 139.7264 126.2236) (end 140.3 125.65) (width 0.25) (layer "B.Cu") (net 33))
   (segment (start 139.8 86.7348) (end 139.1598 87.375) (width 0.2) (layer "B.Cu") (net 39))
   (segment (start 139.1598 87.375) (end 138.525 87.375) (width 0.2) (layer "B.Cu") (net 39))

Commit message: -
Parts:
- moved C6 1.87 mm to (156.2, 91.0)
- moved R5 0.55 mm to (140.6, 101.3)
- moved L2 0.12 mm to (151.3, 93.2)
Routing:
- net Net-(Q1-D): track 33.4 -> 34.7 mm
Changed lines of the file:
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@@
   )
   (footprint "Resistor_SMD:R_0402_1005Metric" (layer "B.Cu")
-    (at 141.15 101.255 90)
+    (at 140.6 101.26 90)
     (descr "Resistor SMD 0402 (1005 Metric), square (rectangular) end terminal, IPC_7351 nominal, (Body size source: IPC-SM-782 page 72, https://www.pcb-3d.com/wordpress/wp-content/uploads/ipc-sm-782a_amendment_1_and_2.pdf), generated with kicad-footprint-generator")
     (tags "resistor")
@@
     (property "ki_keywords" "R res resistor")
     (attr smd)
-    (fp_text reference "R5" (at -0.7768 -1.3484) (layer "B.SilkS")
+    (fp_text reference "R5" (at -0.59 -1.5) (layer "B.SilkS")
         (effects (font (size 1 1) (thickness 0.15)) (justify mirror))
     )
@@
   )
   (footprint "Capacitor_SMD:C_0805_2012Metric" (layer "B.Cu")
-    (at 154.28 91.125)
+    (at 156.15 91)
     (descr "Capacitor SMD 0805 (2012 Metric), square (rectangular) end terminal, IPC_7351 nominal, (Body size source: IPC-SM-782 page 76, https://www.pcb-3d.com/wordpress/wp-content/uploads/ipc-sm-782a_amendment_1_and_2.pdf, https://docs.google.com/spreadsheets/d/1BsfQQcO9C6DZCsRaXUlFlo91Tg2WpOkGARC1WS5S8t0/edit?usp=sharing), generated with kicad-footprint-generator")
     (tags "capacitor")
@@
   )
   (footprint "MAKK2016T1R0M:INDC2016X100N" (layer "B.Cu")
-    (at 151.3752 93.1672)
+    (at 151.253 93.1672)
     (property "Sheetfile" "cm4-gpio.kicad_sch")
     (property "Sheetname" "CM4 GPIO and power pins")
@@
   (segment (start 160.15 93.7) (end 159.275 93.7) (width 0.1524) (layer "B.Cu") (net 6))
   (segment (start 152.575 91.15) (end 152.525 91.1) (width 0.2) (layer "B.Cu") (net 7))
+  (segment (start 155.2 91) (end 155.1 91.1) (width 0.1524) (layer "B.Cu") (net 7))
   (segment (start 152.525 91.1332) (end 152.525 91.1) (width 1) (layer "B.Cu") (net 7))
   (segment (start 147.1175 88.31) (end 147.1175 86.935) (width 0.2) (layer "B.Cu") (net 7))
@@
   (segment (start 153.0858 93.1672) (end 153.8224 92.4306) (width 0.1524) (layer "B.Cu") (net 7))
   (segment (start 152.2222 93.1672) (end 153.0858 93.1672) (width 0.1524) (layer "B.Cu") (net 7))
-  (segment (start 153.975 91.15) (end 152.575 91.15) (width 0.2) (layer "B.Cu") (net 7))
+  (segment (start 155.1 91.1) (end 152.525 91.1) (width 0.1524) (layer "B.Cu") (net 7))
   (segment (start 154.4 100.575) (end 154.35 100.525) (width 1.36703) (layer "B.Cu") (net 7))
   (segment (start 154.4 93.0082) (end 154.4 100.575) (width 1.36703) (layer "B.Cu") (net 7))
@@
   (via (at 141.675 99.55) (size 0.6) (drill 0.3) (layers "F.Cu" "B.Cu") (net 9))
   (via (at 148.55 99.55) (size 0.6) (drill 0.3) (layers "F.Cu" "B.Cu") (net 9))
-  (segment (start 141.15 99.725) (end 140.975 99.55) (width 0.4) (layer "B.Cu") (net 9))
+  (segment (start 140.65 99.875) (end 140.975 99.55) (width 0.4) (layer "B.Cu") (net 9))
   (segment (start 140.975 99.55) (end 138.25 99.55) (width 1.36703) (layer "B.Cu") (net 9))
   (segment (start 149.85 99.55) (end 148.55 99.55) (width 0.2) (layer "B.Cu") (net 9))
   (segment (start 138.25 99.55) (end 138.225 99.525) (width 1.36703) (layer "B.Cu") (net 9))
   (segment (start 141.675 99.55) (end 140.975 99.55) (width 1.36703) (layer "B.Cu") (net 9))
-  (segment (start 141.15 100.95) (end 141.15 99.725) (width 0.4) (layer "B.Cu") (net 9))
+  (segment (start 140.65 100.745) (end 140.65 99.875) (width 0.4) (layer "B.Cu") (net 9))
   (segment (start 147.13 105.4222) (end 147.2946 105.2576) (width 0.4) (layer "B.Cu") (net 10))
   (segment (start 147.13 106.435) (end 144.93 106.435) (width 0.4) (layer "B.Cu") (net 10))
