File: carrier_board_v1.kicad_pcb (KiCad board)
At the start: 2 copper layers, 40.1 x 55.1 mm, 43 parts, among them J1 B2B-PH-SM4-TB_LF__SN_, J3 C262390, J4 C2997432, J5 C2938398, J6 C2997432, Q1 DMP3013SFV, U1 BQ25302RTER, U2 MP28167GQ-P, U3 TPD2EUSB30DRTR

Commit message: complete
Parts:
- removed L1: 4.7uH, Inductor_SMD:L_0805_2012Metric
- added L2: SRP5030CA-2R2M, SRP5030CA-2R2M:SRP5030CA4R7M, B.Cu at (152.3, 104.8)
- C12: value 22nF -> 33nF
- C20: value 10uF -> 100nF
- R5: value 21.5k -> 15k
- moved C4 10.2 mm to (138.2, 94.3), turned to 90 degrees
- moved L3 8.73 mm to (135.7, 96.7), turned to 90 degrees
- moved U2 7.95 mm to (142.6, 104.0)
- moved C9 7.72 mm to (147.5, 106.1)
- moved C10 7.65 mm to (147.5, 102.2)
- moved R1 6.62 mm to (132.8, 86.6)
- moved R2 6.62 mm to (132.8, 88.2)
- moved R7 6.42 mm to (142.2, 108.3)
- moved C17 4.85 mm to (138.6, 91.5)
- moved C3 4.56 mm to (141.9, 95.8), turned to 0 degrees
- moved C14 3.77 mm to (148.0, 109.4), turned to 0 degrees
- moved C13 3.50 mm to (142.2, 109.8), turned to 0 degrees
- moved C16 3.47 mm to (147.0, 113.4), turned to 0 degrees
- moved C6 3.35 mm to (136.3, 104.5), turned to -90 degrees
- moved C15 2.42 mm to (148.0, 110.9), turned to 0 degrees
Routing:
- net Net-(Q1-D): track 25.9 -> 39.3 mm
- net Net-(U1-BAT): track 67.7 -> 79.8 mm, vias 2 -> 5
- net Net-(U1-BTST): track 13.2 -> 2.82 mm, vias 2 -> 0
- net Net-(U1-TS): track 9.10 -> 17.6 mm, vias 0 -> 3
- net Net-(U2-VCC): track 5.25 -> 13.5 mm
- net Net-(U1-SW): track 14.6 -> 7.86 mm, vias 2 -> 0
- net Net-(U2-OC): track 13.4 -> 19.3 mm, vias 0 -> 2
- net +5V: track 108.1 -> 113.1 mm, vias 4 -> 8
- net Net-(U2-SW1): track 6.84 -> 11.7 mm
- net GND: track 0.00 -> 4.41 mm, vias 171 -> 158
- net Net-(U2-SW2): track 6.68 -> 11.1 mm
- net /CM4 GPIO and power pins/REGN: track 22.7 -> 26.7 mm
- net Net-(U1-PMID): track 9.58 -> 6.20 mm
- net Net-(U2-EN): track 7.79 -> 4.77 mm
- net /CM4 GPIO and power pins/GPIO14: track 28.6 -> 25.8 mm
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
Commit message: -
Parts:
- removed D1: CDBA340-HF, Diode_SMD:D_0603_1608Metric
- added J2: DF40C-100DS-0.4V(51), DF40C-100DS-0.4V_51_:HRS_DF40C-100DS-0.4V(51), F.Cu at (120.1, 103.0)
- added J7: DF40C-100DS-0.4V(51), DF40C-100DS-0.4V_51_:HRS_DF40C-100DS-0.4V(51), F.Cu at (170.1, 105.8)
- added U4: CDBA340-HF, CDBA340-HF:CDBA-HF, B.Cu at (154.8, 88.9)
- J1: value B2B-PH-SM4-TB_LF__SN_ -> C157930
- J3: value C262390 -> FH34SRJ-22S-0.5SH50; footprint 54548-2271:MOLEX_54548-2271 -> FH34SRJ-22S-0-5SH-50:CONN22x1_FH34SRJ-22S-0.5SH50_HIR
- R3, R4: value 56kΩ -> 5.1k
- moved R3 6.82 mm to (154.7, 127.2), turned to 180 degrees
- moved R4 6.74 mm to (138.7, 127.2), turned to 0 degrees
- moved J3 1.56 mm to (131.2, 103.5)
- moved J1 0.64 mm to (154.1, 84.1)
- moved C1 0.54 mm to (163.5, 96.9)
- moved J5 0.45 mm to (162.1, 121.1), turned to 0 degrees
Connections:
- J3 pad 18: unconnected-(J3-Pad18) -> GND
- J5 pad 10: /CM4 GPIO and power pins/GPIO10 -> GND
- J5 pad 11: /CM4 GPIO and power pins/GPIO11 -> GND
- J5 pad 13: /CM4 GPIO and power pins/nRPIBOOT -> +3.3V
- J5 pad 14: /CM4 GPIO and power pins/GPIO14 -> +3.3V
- J5 pad 15: /CM4 GPIO and power pins/GPIO15 -> +3.3V
- J5 pad 16: GND -> +3.3V
- J5 pad 4: +3.3V -> /CM4 GPIO and power pins/GPIO4
- J5 pad 5: GND -> /CM4 GPIO and power pins/GPIO5
- J5 pad 6: +3.3V -> /CM4 GPIO and power pins/GPIO6
- J5 pad 7: /CM4 GPIO and power pins/GPIO7 -> /CM4 GPIO and power pins/GPIO27
- J5 pad 8: /CM4 GPIO and power pins/GPIO8 -> GND
- J5 pad 9: /CM4 GPIO and power pins/GPIO9 -> GND
- Module1 pad 30: unconnected-(Module1A-GPIO6-Pad30) -> /CM4 GPIO and power pins/GPIO6
- Module1 pad 34: unconnected-(Module1A-GPIO5-Pad34) -> /CM4 GPIO and power pins/GPIO5
- Module1 pad 37: /CM4 GPIO and power pins/GPIO7 -> unconnected-(Module1A-GPIO7-Pad37)
- Module1 pad 38: /CM4 GPIO and power pins/GPIO11 -> unconnected-(Module1A-GPIO11-Pad38)
- Module1 pad 39: /CM4 GPIO and power pins/GPIO8 -> unconnected-(Module1A-GPIO8-Pad39)
- Module1 pad 40: /CM4 GPIO and power pins/GPIO9 -> unconnected-(Module1A-GPIO9-Pad40)
- Module1 pad 44: /CM4 GPIO and power pins/GPIO10 -> unconnected-(Module1A-GPIO10-Pad44)
- Module1 pad 48: unconnected-(Module1A-GPIO27-Pad48) -> /CM4 GPIO and power pins/GPIO27
- Module1 pad 51: /CM4 GPIO and power pins/GPIO15 -> unconnected-(Module1A-GPIO15-Pad51)
- Module1 pad 54: unconnected-(Module1A-GPIO4-Pad54) -> /CM4 GPIO and power pins/GPIO4
- Module1 pad 55: /CM4 GPIO and power pins/GPIO14 -> unconnected-(Module1A-GPIO14-Pad55)
- Module1 pad 93: /CM4 GPIO and power pins/nRPIBOOT -> unconnected-(Module1A-nRPIBOOT-Pad93)
- R3 pad 1: +5V -> GND
- R4 pad 1: +5V -> GND
Routing:
- net /CM4 GPIO and power pins/nRPIBOOT: track 51.3 -> 0.00 mm, vias 5 -> 0
- net /CM4 GPIO and power pins/GPIO10: track 34.5 -> 0.00 mm, vias 1 -> 0
- net /CM4 GPIO and power pins/GPIO27: track 0.00 -> 28.7 mm, vias 0 -> 1
- net /CM4 GPIO and power pins/GPIO4: track 0.00 -> 26.7 mm, vias 0 -> 1
- net /CM4 GPIO and power pins/GPIO14: track 25.8 -> 0.00 mm, vias 1 -> 0
- net /CM4 GPIO and power pins/GPIO15: track 24.8 -> 0.00 mm, vias 1 -> 0
- net /CM4 GPIO and power pins/GPIO5: track 0.00 -> 23.7 mm, vias 0 -> 1
- net /CM4 GPIO and power pins/GPIO11: track 23.1 -> 0.00 mm, vias 1 -> 0
- net /CM4 GPIO and power pins/GPIO6: track 0.00 -> 22.4 mm, vias 0 -> 1
- net /CM4 GPIO and power pins/GPIO9: track 22.0 -> 0.00 mm, vias 1 -> 0
- net /CM4 GPIO and power pins/GPIO7: track 20.7 -> 0.00 mm, vias 1 -> 0
- net /CM4 GPIO and power pins/GPIO8: track 17.1 -> 0.00 mm, vias 1 -> 0
- net /CM4 GPIO and power pins/GPIO3: track 19.0 -> 36.1 mm
- net /CM4 GPIO and power pins/GPIO2: track 16.1 -> 30.3 mm
- net GND: track 4.41 -> 17.8 mm, vias 158 -> 127
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
Commit message: -
Parts:
- moved J7 21.8 mm to (191.4, 101.2)
- moved J2 15.8 mm to (104.5, 100.7)
Connections:
- J4 pad S1: Net-(J4-SHELL_GND-PadS1) -> GND
- J4 pad S2: Net-(J4-SHELL_GND-PadS1) -> GND
- J4 pad S3: Net-(J4-SHELL_GND-PadS1) -> GND
- J4 pad S4: Net-(J4-SHELL_GND-PadS1) -> GND
Routing:
- net Net-(J4-SHELL_GND-PadS1): track 17.0 -> 0.00 mm
- net +5V: track 102.0 -> 101.1 mm, vias 8 -> 7
- net /CM4 GPIO and power pins/GPIO5: track 23.7 -> 24.6 mm
- net Net-(Q1-D): track 39.0 -> 38.4 mm
- net SDA0: track 55.4 -> 55.3 mm, vias 4 -> 3
- net SCL0: vias 2 -> 1
- net GND: vias 127 -> 135
- net CAM_GPIO: vias 2 -> 1

Commit message: -
Parts:
- removed C15: 22uF, Capacitor_SMD:C_0603_1608Metric
- removed C16: 100uF, Capacitor_Tantalum_SMD:CP_EIA-3528-21_Kemet-B
- removed C17: 2.2uF, Capacitor_SMD:C_0603_1608Metric
- removed C18, C19: 10uF, Capacitor_SMD:C_0603_1608Metric
- removed C20: 100nF, Capacitor_SMD:C_0603_1608Metric
- removed L3: 1uH, Inductor_SMD:L_0805_2012Metric
- removed U1: BQ25302RTER, BQ25302:RTE0016C
- removed U4: CDBA340-HF, CDBA340-HF:CDBA-HF
- added IC1: LTC4413EDD-1#PBF, LTC4413EDD_PBF:SON50P300X300X80-11N, B.Cu at (155.9, 91.5)
- added L1: 1uH, Inductor_SMD:L_0805_2012Metric, B.Cu at (143.5, 97.9)
- added R11: 61.9k, Resistor_SMD:R_0603_1608Metric, B.Cu at (152.0, 105.7)
- added R8: 1M, Resistor_SMD:R_0603_1608Metric, B.Cu at (148.9, 107.2)
- added U7: BQ25302RTER, BQ25302:RTE0016C, B.Cu at (148.8, 93.6)
- C1: value 100uF -> 10uF; footprint Capacitor_Tantalum_SMD:CP_EIA-3528-21_Kemet-B -> Capacitor_SMD:C_0603_1608Metric
- C10: value 100nF -> 10uF
- C11: value 1uF -> 47uF
- C12: value 33nF -> 2.2uF
- C13: value 22nF -> 10uF
- C14, C8: value 0.1uF -> 10uF
- C9: value 100nF -> 1uF
- R1, R2: value 10kΩ -> 10k
- R10: value 23.2kΩ -> 23.2k
- R5: value 15k -> 332k
- R7: value 499kΩ -> 1M
- U2: value MP28167GQ-P -> TPS61235PRWLT; footprint MP28167GQ-P:QFN-16_MP28167GQ_MNP -> TPS61235PRWLT:RWL0009A
- moved R10 32.6 mm to (115.9, 85.3)
- moved C12 31.1 mm to (119.9, 84.7), turned to 180 degrees
- moved C13 28.7 mm to (160.7, 87.9), turned to 90 degrees
- moved C5 26.2 mm to (121.1, 87.8), turned to 180 degrees
- moved C14 25.8 mm to (162.2, 87.9), turned to 90 degrees
- moved C3 25.4 mm to (119.9, 83.1), turned to 180 degrees
- moved R1 21.4 mm to (111.6, 83.4)
- moved R2 21.3 mm to (111.6, 85.9), turned to 180 degrees
- moved J7 21.2 mm to (170.3, 102.2)
- moved C4 20.1 mm to (119.9, 86.2), turned to 0 degrees
- moved J2 18.8 mm to (123.0, 103.7)
- moved R5 17.2 mm to (140.7, 110.5), turned to 180 degrees
- moved C1 13.6 mm to (152.0, 104.1), turned to 180 degrees
- moved C8 13.3 mm to (152.0, 107.2), turned to 180 degrees
- moved C6 12.4 mm to (143.6, 94.5), turned to 0 degrees
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Connections:
- C1 pad 1: Net-(Q1-D) -> Net-(IC1-INA)
- C10 pad 1: Net-(U2-SW2) -> Net-(Q1-D)
- C10 pad 2: Net-(U2-BST2) -> GND
- C11 pad 1: GND -> Net-(Q1-D)
- C11 pad 2: Net-(U2-VCC) -> GND
- C12 pad 1: Net-(U2-OC) -> Net-(U7-PMID)
- C13 pad 1: Net-(U2-EN) -> +5V
- C14 pad 1: Net-(U1-BAT) -> +5V
- C2 pad 1: Net-(Q1-D) -> Net-(IC1-INA)
- C6 pad 1: Net-(U1-BAT) -> Net-(U7-BAT)
- C7 pad 1: Net-(Q1-D) -> Net-(IC1-INA)
- C8 pad 1: Net-(Q1-D) -> Net-(U2-CC)
- C9 pad 1: Net-(U2-SW1) -> Net-(Q1-D)
- C9 pad 2: Net-(U2-BST1) -> GND
- J1 pad 2: Net-(U1-BAT) -> Net-(U7-BAT)
- L2 pad 1: Net-(U2-SW1) -> Net-(U2-SW)
- L2 pad 2: Net-(U2-SW2) -> Net-(Q1-D)
- Q1 pad 1: +5V -> Net-(U7-BAT)
- Q1 pad 2: +5V -> Net-(U7-BAT)
- Q1 pad 3: +5V -> Net-(U7-BAT)
- R1 pad 1: Net-(U1-TS) -> GND
- R1 pad 2: /CM4 GPIO and power pins/REGN -> Net-(U7-TS)
- R10 pad 1: GND -> Net-(U7-ICHG)
- R10 pad 2: Net-(U1-ICHG_EN) -> GND
- R2 pad 1: GND -> /CM4 GPIO and power pins/REGN
- R2 pad 2: Net-(U1-TS) -> Net-(U7-TS)
- R5 pad 1: GND -> Net-(U2-FB)
- R5 pad 2: Net-(U2-OC) -> GND
- R7 pad 1: Net-(U2-EN) -> Net-(IC1-INA)
- R7 pad 2: Net-(U1-BAT) -> Net-(U2-FB)
- U2 pad 1: Net-(U1-BAT) -> GND
- U2 pad 2: GND -> Net-(U2-SW)
- U2 pad 3: Net-(U2-EN) -> Net-(Q1-D)
- U2 pad 4: unconnected-(U2-NC-Pad4) -> Net-(U2-CC)
- U2 pad 6: GND -> Net-(U2-FB)
- U2 pad 7: Net-(U2-OC) -> Net-(U2-EN)
- U2 pad 9: Net-(U2-VCC) -> Net-(IC1-INA)
Routing:
- net Net-(U1-BAT): track 87.8 -> 0.00 mm, vias 5 -> 0
- net Net-(IC1-INA): track 0.00 -> 39.9 mm
- net Net-(IC1-INB): track 62.5 -> 33.9 mm, vias 4 -> 0
- net Net-(U7-BAT): track 0.00 -> 27.3 mm, vias 0 -> 4
- net /CM4 GPIO and power pins/REGN: track 26.7 -> 0.01 mm, vias 2 -> 0
- net Net-(U2-OC): track 19.3 -> 0.00 mm, vias 2 -> 0
- net Net-(U1-TS): track 17.1 -> 0.00 mm, vias 2 -> 0
- net Net-(Q1-D): track 38.4 -> 21.8 mm, vias 2 -> 0
- net +5V: track 101.1 -> 85.5 mm
- net Net-(U2-VCC): track 13.5 -> 0.00 mm
- net Net-(U2-SW1): track 11.7 -> 0.00 mm
- net Net-(U2-SW2): track 11.1 -> 0.00 mm
- net Net-(U2-CC): track 0.00 -> 10.6 mm
- net Net-(U2-FB): track 0.00 -> 10.3 mm, vias 0 -> 2
- net Net-(U7-BTST): track 7.86 -> 0.00 mm
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
Commit message: version3 complete
Parts:
- C1, C2, C7: value 10uF -> 22uF
- C11: footprint Capacitor_SMD:C_0603_1608Metric -> Capacitor_SMD:C_1206_3216Metric
- L2: value SRP5030CA-2R2M -> MDMK4040T1R0MM; footprint SRP5030CA-2R2M:SRP5030CA4R7M -> MDMK4040T1R0MM:MDMK4040T1R0MM
- R10: value 23.2k -> 40.2k
- moved R1 42.8 mm to (153.4, 92.6)
- moved R2 42.0 mm to (152.7, 94.9), turned to 90 degrees
- moved R10 37.2 mm to (152.7, 90.2), turned to 0 degrees
- moved C5 33.1 mm to (152.0, 99.5)
- moved C3 30.6 mm to (149.7, 90.2), turned to 0 degrees
- moved C4 24.5 mm to (143.5, 92.9)
- moved C12 24.5 mm to (143.5, 91.4)
- moved C6 6.03 mm to (138.4, 97.4), turned to -90 degrees
- moved C11 5.56 mm to (138.3, 100.2)
- moved C10 4.86 mm to (139.0, 102.2)
- moved L1 4.35 mm to (140.7, 94.5), turned to 0 degrees
- moved Q1 3.52 mm to (144.1, 99.1)
- moved IC1 2.41 mm to (158.3, 91.2)
- moved C13 0.62 mm to (161.3, 87.9)
- moved C14 0.62 mm to (162.8, 87.9)
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Connections:
- R8 pad 2: Net-(U2-EN) -> GND
- U2 pad 7: Net-(U2-EN) -> Net-(Q1-D)
Routing:
- net Net-(IC1-INB): track 33.9 -> 54.3 mm, vias 0 -> 2
- net Net-(Q1-D): track 21.8 -> 39.5 mm, vias 0 -> 2
- net Net-(U7-BAT): track 27.3 -> 45.1 mm
- net /CM4 GPIO and power pins/REGN: track 0.01 -> 13.2 mm, vias 0 -> 2
- net Net-(C4-Pad1): track 0.00 -> 9.25 mm
- net Net-(U2-SW): track 0.00 -> 6.63 mm
- net Net-(U2-EN): track 6.45 -> 0.00 mm, vias 2 -> 0
- net Net-(U7-TS): track 0.00 -> 5.57 mm
- net Net-(U7-ICHG): track 0.00 -> 4.31 mm
- net Net-(U7-PMID): track 0.00 -> 4.13 mm
- net +5V: track 85.5 -> 81.4 mm
- net Net-(U7-BTST): track 0.00 -> 3.27 mm
- net SCL0: track 56.3 -> 54.0 mm
- net (no net): track 2.27 -> 0.00 mm, vias 1 -> 0
- net Net-(U2-FB): track 10.3 -> 12.4 mm
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