File: cm4-gpio.kicad_sch (KiCad schematic)
At the start: 26 parts, among them J1 B2B-PH-SM4-TB_LF__SN_, J6 USB4105-GF-A, J7 Conn_01x12_Pin, Q1 DMP3013SFV, U1 BQ25302RTER, U5 TPS613222ADBZ

Commit message: -
Changed lines of the file:
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@@
   (no_connect (at 158.115 119.38))
   (no_connect (at 241.935 202.565))
-  (wire (pts (xy 81.28 223.52) (xy 95.885 223.52))
+  (wire (pts (xy 80.645 223.52) (xy 95.885 223.52))
     (stroke (width 0) (type default))
   )
@@
     )
   )
-  (global_label "+1.8V" (shape output) (at 81.28 223.52 180)
+  (global_label "+1.8V" (shape output) (at 80.645 223.52 180)
     (effects (font (size 1.27 1.27)) (justify right))
-    (property "Intersheetrefs" "${INTERSHEET_REFS}" (at 81.28 223.52 0)
+    (property "Intersheetrefs" "${INTERSHEET_REFS}" (at 80.645 223.52 0)
       (effects (font (size 1.27 1.27)) hide)
     )

Commit message: -
Connections:
- net +1.8V: no longer names the net of Module1.88 (+1.8v_(Output))
- net +1.8V: no longer Module1.90 (+1.8v_(Output))
- no-connect marks 64 -> 66
Changed lines of the file:
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@@
   (junction (at 94.615 139.7) (diameter 1.016) (color 0 0 0 0)
-  )
-  (junction (at 95.885 223.52) (diameter 0) (color 0 0 0 0)
   )
   (junction (at 94.615 205.74) (diameter 1.016) (color 0 0 0 0)
@@
   (no_connect (at 158.115 127))
   (no_connect (at 158.115 170.18))
+  (no_connect (at 97.155 223.52))
   (no_connect (at 241.935 200.025))
   (no_connect (at 158.115 185.42))
@@
   (no_connect (at 158.115 152.4))
   (no_connect (at 158.115 205.74))
+  (no_connect (at 97.155 226.06))
   (no_connect (at 97.155 200.66))
   (no_connect (at 158.115 147.32))
@@
   (no_connect (at 158.115 119.38))
   (no_connect (at 241.935 202.565))
-  (wire (pts (xy 80.645 223.52) (xy 95.885 223.52))
-    (stroke (width 0) (type default))
-  )
   (wire (pts (xy 408.94 282.575) (xy 436.88 282.575))
     (stroke (width 0) (type default))
@@
     (stroke (width 0) (type solid))
   )
-  (wire (pts (xy 95.885 226.06) (xy 95.885 223.52))
-    (stroke (width 0) (type solid))
-  )
   (wire (pts (xy 158.115 182.88) (xy 163.195 182.88))
     (stroke (width 0) (type default))
@@
     (stroke (width 0) (type solid))
   )
-  (wire (pts (xy 97.155 226.06) (xy 95.885 226.06))
-    (stroke (width 0) (type solid))
-  )
   (wire (pts (xy 94.615 139.7) (xy 94.615 152.4))
     (stroke (width 0) (type solid))
@@
   )
   (wire (pts (xy 94.615 187.96) (xy 97.155 187.96))
-    (stroke (width 0) (type solid))
-  )
-  (wire (pts (xy 95.885 223.52) (xy 97.155 223.52))
     (stroke (width 0) (type solid))
   )
@@
     )
   )
-  (global_label "+1.8V" (shape output) (at 80.645 223.52 180)
-    (effects (font (size 1.27 1.27)) (justify right))
-    (property "Intersheetrefs" "${INTERSHEET_REFS}" (at 80.645 223.52 0)
-      (effects (font (size 1.27 1.27)) hide)
-    )
-  )

Commit message: -
Parts:
- removed L1: 2.2u, Inductor_SMD:L_0201_0603Metric, symbol dk_Fixed-Inductors:13R106C
- removed L2: 1u, Inductor_SMD:L_0201_0603Metric, symbol dk_Fixed-Inductors:13R106C
- added L1: 1.5uH, Inductor_SMD:L_1008_2520Metric, symbol dk_Fixed-Inductors:82473C
- added L2: MAKK2016T1R0M, INDC2016X100N, symbol MAKK2016T1R0M:MAKK2016T1R0M
- C1: value 22u -> 22uF; footprint Capacitor_SMD:C_0201_0603Metric -> Capacitor_SMD:C_0603_1608Metric
- C2, C6: value 10u -> 10uF; footprint Capacitor_SMD:C_0201_0603Metric -> Capacitor_SMD:C_0805_2012Metric
- C3, C8: value 2.2u -> 2.2uF; footprint Capacitor_SMD:C_0201_0603Metric -> Capacitor_SMD:C_0603_1608Metric
- C4: value 47n -> 47nF; footprint Capacitor_SMD:C_0201_0603Metric -> Capacitor_SMD:C_0603_1608Metric
- C5: footprint Capacitor_SMD:C_0201_0603Metric -> Capacitor_SMD:C_0603_1608Metric
- R1: value 4.527 -> 4.53; footprint Resistor_SMD:R_0201_0603Metric -> Resistor_SMD:R_1206_3216Metric
- R10: value 20k -> 20kΩ; footprint Resistor_SMD:R_0201_0603Metric -> Resistor_SMD:R_0402_1005Metric
- R2: value 23.26 -> 22; footprint Resistor_SMD:R_0201_0603Metric -> Resistor_SMD:R_0805_2012Metric
- R5: value 1 -> 1.1; footprint Resistor_SMD:R_0201_0603Metric -> Resistor_SMD:R_0402_1005Metric
- R6, R9: value 5.1k -> 5.1kΩ; footprint Resistor_SMD:R_0201_0603Metric -> Resistor_SMD:R_0402_1005Metric
Connections:
- net PMID: now also L1.2
- net at C4.2, U1.13 (SW): now also L2.1
- net at C6.1, J1.2, Q1.5 (D)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: now also L2.2
- net at D2.2 (A), U5.2 (SW): now also L1.1
Other:
- moved on the sheet: C8

Commit message: -
Parts:
- removed U5: TPS613222ADBZ, Package_TO_SOT_SMD:SOT-23, symbol Regulator_Switching:TPS613222ADBZ
- added U2: TPS613222ADBVT, SOT95P280X145-5N, symbol TPS613222ADBVT:TPS613222ADBVT
Connections:
- net +5V: now also U2.4 (VOUT)
- net GND: now also U2.2 (GND)
- net at D2.2 (A), L1.1: now also U2.1 (SW)
Other:
- moved on the sheet: C1
Changed lines of the file:
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@@
   (junction (at 94.615 205.74) (diameter 1.016) (color 0 0 0 0)
   )
+  (junction (at 293.37 132.08) (diameter 0) (color 0 0 0 0)
+  )
   (junction (at 160.655 154.94) (diameter 1.016) (color 0 0 0 0)
   )
@@
   (junction (at 159.385 213.36) (diameter 1.016) (color 0 0 0 0)
   )
-  (junction (at 293.37 132.08) (diameter 0) (color 0 0 0 0)
-  )
   (junction (at 160.655 129.54) (diameter 1.016) (color 0 0 0 0)
   )
@@
   (junction (at 436.88 282.575) (diameter 0) (color 0 0 0 0)
   )
-  (junction (at 252.095 132.08) (diameter 0) (color 0 0 0 0)
+  (junction (at 234.95 132.08) (diameter 0) (color 0 0 0 0)
   )
   (junction (at 423.545 139.065) (diameter 0) (color 0 0 0 0)
@@
     (stroke (width 0) (type default))
   )
-  (wire (pts (xy 252.095 116.84) (xy 252.095 132.08))
-    (stroke (width 0) (type default))
-  )
-  (wire (pts (xy 269.875 116.84) (xy 252.095 116.84))
+  (wire (pts (xy 234.95 116.84) (xy 234.95 132.08))
+    (stroke (width 0) (type default))
+  )
+  (wire (pts (xy 269.875 116.84) (xy 234.95 116.84))
     (stroke (width 0) (type default))
   )
@@
     (stroke (width 0) (type solid))
   )
-  (wire (pts (xy 283.845 132.08) (xy 293.37 132.08))
-    (stroke (width 0) (type default))
-  )
   (wire (pts (xy 409.575 267.97) (xy 436.88 267.97))
     (stroke (width 0) (type default))
@@
     (stroke (width 0) (type solid))
   )
-  (wire (pts (xy 201.295 132.08) (xy 252.095 132.08))
+  (wire (pts (xy 184.15 132.08) (xy 234.95 132.08))
     (stroke (width 0) (type default))
   )
@@
     (stroke (width 0) (type solid))
   )
-  (wire (pts (xy 159.385 210.82) (xy 201.295 210.82))
+  (wire (pts (xy 159.385 210.82) (xy 184.15 210.82))
     (stroke (width 0) (type solid))
   )
@@
     (stroke (width 0) (type default))
   )
-  (wire (pts (xy 252.095 132.08) (xy 263.525 132.08))
-    (stroke (width 0) (type default))
-  )
   (wire (pts (xy 454.025 154.94) (xy 454.025 152.4))
     (stroke (width 0) (type default))
@@
     (stroke (width 0) (type default))
   )
+  (wire (pts (xy 248.92 132.08) (xy 234.95 132.08))
+    (stroke (width 0) (type default))
+  )
   (wire (pts (xy 454.025 152.4) (xy 462.915 152.4))
     (stroke (width 0) (type default))
@@
     (stroke (width 0) (type solid))
   )
-  (wire (pts (xy 252.095 141.605) (xy 252.095 144.78))
-    (stroke (width 0) (type default))
-  )
-  (wire (pts (xy 252.095 133.985) (xy 252.095 132.08))
+  (wire (pts (xy 234.95 141.605) (xy 234.95 144.78))
+    (stroke (width 0) (type default))
+  )
+  (wire (pts (xy 234.95 133.985) (xy 234.95 132.08))
     (stroke (width 0) (type default))
   )
@@
     (stroke (width 0) (type solid))
   )
-  (wire (pts (xy 201.295 132.08) (xy 201.295 210.82))
-    (stroke (width 0) (type default))
-  )
-  (wire (pts (xy 273.685 142.24) (xy 273.685 144.78))
+  (wire (pts (xy 184.15 132.08) (xy 184.15 210.82))
+    (stroke (width 0) (type default))
+  )
+  (wire (pts (xy 251.46 127) (xy 257.81 127))
     (stroke (width 0) (type default))
   )
@@
     (stroke (width 0) (type default))
   )
+  (wire (pts (xy 257.81 137.16) (xy 248.92 137.16))
+    (stroke (width 0) (type default))
+  )
   (wire (pts (xy 135.255 307.34) (xy 125.095 307.34))
     (stroke (width 0) (type solid))
@@
   (wire (pts (xy 94.615 165.1) (xy 94.615 177.8))
     (stroke (width 0) (type solid))
+  )
+  (wire (pts (xy 248.92 137.16) (xy 248.92 132.08))
+    (stroke (width 0) (type default))
   )
   (wire (pts (xy 464.82 192.405) (xy 464.82 222.885))
@@
     )
   )
-  (symbol (lib_name "GND_6") (lib_id "power:GND") (at 252.095 144.78 0) (unit 1)
-    (in_bom yes) (on_board yes) (dnp no) (fields_autoplaced)
-    (property "Reference" "#PWR04" (at 252.095 151.13 0)
-      (effects (font (size 1.27 1.27)) hide)
-    )
-    (property "Value" "GND" (at 252.095 149.86 0)
-      (effects (font (size 1.27 1.27)))
-    )
-    (property "Footprint" "" (at 252.095 144.78 0)
-      (effects (font (size 1.27 1.27)) hide)
-    )
-    (property "Datasheet" "" (at 252.095 144.78 0)
+  (symbol (lib_name "GND_6") (lib_id "power:GND") (at 234.95 144.78 0) (unit 1)
+    (in_bom yes) (on_board yes) (dnp no) (fields_autoplaced)
+    (property "Reference" "#PWR04" (at 234.95 151.13 0)
+      (effects (font (size 1.27 1.27)) hide)
+    )
+    (property "Value" "GND" (at 234.95 149.86 0)
+      (effects (font (size 1.27 1.27)))
+    )
+    (property "Footprint" "" (at 234.95 144.78 0)
+      (effects (font (size 1.27 1.27)) hide)
+    )
+    (property "Datasheet" "" (at 234.95 144.78 0)
       (effects (font (size 1.27 1.27)) hide)
     )
@@
     )
   )
-  (symbol (lib_id "Device:C") (at 252.095 137.795 0) (unit 1)
-    (in_bom yes) (on_board yes) (dnp no) (fields_autoplaced)
-    (property "Reference" "C1" (at 255.27 136.525 0)
+  (symbol (lib_id "Device:C") (at 234.95 137.795 0) (unit 1)
+    (in_bom yes) (on_board yes) (dnp no) (fields_autoplaced)
+    (property "Reference" "C1" (at 238.125 136.525 0)
       (effects (font (size 1.27 1.27)) (justify left))
     )
-    (property "Value" "22uF" (at 255.27 139.065 0)
+    (property "Value" "22uF" (at 238.125 139.065 0)
       (effects (font (size 1.27 1.27)) (justify left))
     )
-    (property "Footprint" "Capacitor_SMD:C_0603_1608Metric" (at 253.0602 141.605 0)
-      (effects (font (size 1.27 1.27)) hide)
-    )
-    (property "Datasheet" "~" (at 252.095 137.795 0)
+    (property "Footprint" "Capacitor_SMD:C_0603_1608Metric" (at 235.9152 141.605 0)
+      (effects (font (size 1.27 1.27)) hide)
+    )
+    (property "Datasheet" "~" (at 234.95 137.795 0)
       (effects (font (size 1.27 1.27)) hide)
     )
@@
     )
   )
+  (symbol (lib_id "TPS613222ADBVT:TPS613222ADBVT") (at 275.59 132.08 180) (unit 1)
+    (in_bom yes) (on_board yes) (dnp no) (fields_autoplaced)
+    (property "Reference" "U2" (at 275.59 119.38 0)
+      (effects (font (size 1.27 1.27)))
+    )
+    (property "Value" "TPS613222ADBVT" (at 275.59 121.92 0)
+      (effects (font (size 1.27 1.27)))
+    )
+    (property "Footprint" "SOT95P280X145-5N" (at 275.59 132.08 0)
+      (effects (font (size 1.27 1.27)) (justify bottom) hide)
+    )
+    (property "Datasheet" "" (at 275.59 132.08 0)
+      (effects (font (size 1.27 1.27)) hide)
+    )
+    (pin "1")
+    (pin "2")
+    (pin "4")
+    (instances
+      (project "carrier_board_v1"
+        (path "/7c2e4356-99de-4c13-89ad-ca928a2db042/fc4c71a5-1008-4ac4-98db-57c838c57d91"
+          (reference "U2") (unit 1)
+        )
+      )
+    )
+  )
   (symbol (lib_name "GND_1") (lib_id "power:GND") (at 332.105 200.025 0) (unit 1)
     (in_bom yes) (on_board yes) (dnp no) (fields_autoplaced)
@@
         (path "/7c2e4356-99de-4c13-89ad-ca928a2db042/fc4c71a5-1008-4ac4-98db-57c838c57d91"
           (reference "#PWR02") (unit 1)
-        )
-      )
-    )
-  )
-  (symbol (lib_id "Regulator_Switching:TPS613222ADBZ") (at 273.685 134.62 0) (mirror y) (unit 1)
-    (in_bom yes) (on_board yes) (dnp no)
-    (property "Reference" "U5" (at 273.685 124.46 0)
-      (effects (font (size 1.27 1.27)))
-    )
-    (property "Value" "TPS613222ADBZ" (at 273.685 127 0)
-      (effects (font (size 1.27 1.27)))
-    )
-    (property "Footprint" "Package_TO_SOT_SMD:SOT-23" (at 273.685 154.94 0)
-      (effects (font (size 1.27 1.27)) hide)
-    )
-    (property "Datasheet" "http://www.ti.com/lit/ds/symlink/tps61322.pdf" (at 273.685 138.43 0)
-      (effects (font (size 1.27 1.27)) hide)
-    )
-    (pin "1")
-    (pin "2")
-    (pin "3")
-    (instances
-      (project "carrier_board_v1"
-        (path "/7c2e4356-99de-4c13-89ad-ca928a2db042/fc4c71a5-1008-4ac4-98db-57c838c57d91"
-          (reference "U5") (unit 1)
         )
       )
@@
     )
   )
-  (symbol (lib_name "GND_6") (lib_id "power:GND") (at 273.685 144.78 0) (unit 1)
-    (in_bom yes) (on_board yes) (dnp no) (fields_autoplaced)
-    (property "Reference" "#PWR01" (at 273.685 151.13 0)
-      (effects (font (size 1.27 1.27)) hide)
-    )
-    (property "Value" "GND" (at 273.685 149.86 0)
-      (effects (font (size 1.27 1.27)))
-    )
-    (property "Footprint" "" (at 273.685 144.78 0)
-      (effects (font (size 1.27 1.27)) hide)
-    )
-    (property "Datasheet" "" (at 273.685 144.78 0)
-      (effects (font (size 1.27 1.27)) hide)
-    )
+  (symbol (lib_name "GND_6") (lib_id "power:GND") (at 251.46 127 270) (unit 1)
+    (in_bom yes) (on_board yes) (dnp no) (fields_autoplaced)
+    (property "Reference" "#PWR01" (at 245.11 127 0)
+      (effects (font (size 1.27 1.27)) hide)
+    )
+    (property "Value" "GND" (at 246.38 127 0)
+      (effects (font (size 1.27 1.27)))
+    )
+    (property "Footprint" "" (at 251.46 127 0)
+      (effects (font (size 1.27 1.27)) hide)
+    )
+    (property "Datasheet" "" (at 251.46 127 0)
+      (effects (font (size 1.27 1.27)) hide)
+    )
