File: cm4-gpio.kicad_sch (KiCad schematic)
At the start: 25 parts, among them J1 B2B-PH-SM4-TB_LF__SN_, J6 USB4105-GF-A, J7 Conn_01x12_Pin, Q1 DMP3013SFV, U1 BQ25302RTER, U2 TPS61256YFFR

Commit message: final commit
Parts:
- C6: footprint Capacitor_SMD:C_0805_2012Metric -> Capacitor_SMD:C_0603_1608Metric
- R5: footprint Resistor_SMD:R_0402_1005Metric -> Resistor_SMD:R_0603_1608Metric
Connections:
- net PMID: now also U2.B3 (EN)
Changed lines of the file:
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@@
   (junction (at 248.285 131.445) (diameter 0) (color 0 0 0 0)
+  )
+  (junction (at 314.96 123.825) (diameter 0) (color 0 0 0 0)
   )
   (junction (at 159.385 210.82) (diameter 0) (color 0 0 0 0)
@@
     (stroke (width 0) (type default))
   )
+  (wire (pts (xy 302.26 146.685) (xy 314.96 146.685))
+    (stroke (width 0) (type default))
+  )
   (wire (pts (xy 231.775 197.485) (xy 231.775 198.755))
     (stroke (width 0) (type default))
@@
     (stroke (width 0) (type default))
   )
+  (wire (pts (xy 314.96 123.825) (xy 327.025 123.825))
+    (stroke (width 0) (type default))
+  )
   (wire (pts (xy 158.115 160.02) (xy 162.56 160.02))
     (stroke (width 0) (type default))
@@
     (stroke (width 0) (type default))
   )
+  (wire (pts (xy 314.96 146.685) (xy 314.96 123.825))
+    (stroke (width 0) (type default))
+  )
   (wire (pts (xy 318.77 207.645) (xy 353.06 207.645))
     (stroke (width 0) (type default))
@@
     (stroke (width 0) (type default))
   )
-  (wire (pts (xy 306.705 123.825) (xy 327.025 123.825))
+  (wire (pts (xy 306.705 123.825) (xy 314.96 123.825))
     (stroke (width 0) (type default))
   )
@@
       (effects (font (size 1.27 1.27)) (justify left))
     )
-    (property "Footprint" "Capacitor_SMD:C_0805_2012Metric" (at 452.4502 200.025 0)
+    (property "Footprint" "Capacitor_SMD:C_0603_1608Metric" (at 452.4502 200.025 0)
       (effects (font (size 1.27 1.27)) hide)
     )
@@
       (effects (font (size 1.27 1.27)) (justify right))
     )
-    (property "Footprint" "Resistor_SMD:R_0402_1005Metric" (at 455.803 158.75 90)
-      (effects (font (size 1.27 1.27)) hide)
-    )
+    (property "Footprint" "Resistor_SMD:R_0603_1608Metric" (at 455.803 158.75 90)
+      (effects (font (size 1.27 1.27)) hide)
+    )

Commit message: no
Connections:
- net +5V: no longer C3.1, CR1.1, D1.2 (A), J6.A4_B9 (VBUS), J6.B4_A9 (VBUS), U1.16 (VBUS)
- new net VBUS: C3.1, CR1.1, D1.2 (A), J6.A4_B9 (VBUS), J6.B4_A9 (VBUS), U1.16 (VBUS)
Changed lines of the file:
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@@
   (junction (at 400.685 207.645) (diameter 0) (color 0 0 0 0)
   )
+  (junction (at 438.785 139.065) (diameter 0) (color 0 0 0 0)
+  )
   (junction (at 160.655 180.34) (diameter 1.016) (color 0 0 0 0)
   )
@@
   )
   (junction (at 160.655 195.58) (diameter 1.016) (color 0 0 0 0)
-  )
-  (junction (at 438.785 139.065) (diameter 0) (color 0 0 0 0)
   )
   (junction (at 159.385 213.36) (diameter 1.016) (color 0 0 0 0)
@@
     (stroke (width 0) (type solid))
   )
+  (wire (pts (xy 438.785 123.825) (xy 438.785 139.065))
+    (stroke (width 0) (type default))
+  )
   (wire (pts (xy 423.545 139.065) (xy 438.785 139.065))
     (stroke (width 0) (type default))
@@
     (stroke (width 0) (type default))
   )
-  (wire (pts (xy 190.5 131.445) (xy 236.855 131.445))
-    (stroke (width 0) (type default))
-  )
   (wire (pts (xy 314.96 146.685) (xy 314.96 123.825))
     (stroke (width 0) (type default))
@@
     (stroke (width 0) (type default))
   )
-  (wire (pts (xy 438.785 139.065) (xy 438.785 123.825))
-    (stroke (width 0) (type default))
-  )
   (wire (pts (xy 135.255 292.1) (xy 125.095 292.1))
     (stroke (width 0) (type solid))
@@
     (stroke (width 0) (type default))
   )
+  (wire (pts (xy 327.025 123.825) (xy 438.785 123.825))
+    (stroke (width 0) (type default))
+  )
   (wire (pts (xy 94.615 139.7) (xy 94.615 152.4))
     (stroke (width 0) (type solid))
@@
     (stroke (width 0) (type default))
   )
-  (wire (pts (xy 327.025 123.825) (xy 438.785 123.825))
-    (stroke (width 0) (type default))
-  )
   (wire (pts (xy 306.705 123.825) (xy 314.96 123.825))
     (stroke (width 0) (type default))
@@
     (stroke (width 0) (type solid))
   )
-  (wire (pts (xy 190.5 131.445) (xy 190.5 210.82))
-    (stroke (width 0) (type default))
-  )
   (wire (pts (xy 284.48 212.725) (xy 284.48 215.265))
     (stroke (width 0) (type default))
@@
   )
   (wire (pts (xy 87.63 167.64) (xy 97.155 167.64))
+    (stroke (width 0) (type default))
+  )
+  (wire (pts (xy 219.075 131.445) (xy 236.855 131.445))
     (stroke (width 0) (type default))
   )
@@
     (effects (font (size 1.27 1.27)) (justify right bottom))
   )
+  (label "VBUS" (at 485.14 152.4 0) (fields_autoplaced)
+    (effects (font (size 1.27 1.27)) (justify left bottom))
+  )
+  (label "VSYS" (at 190.5 210.82 0) (fields_autoplaced)
+    (effects (font (size 1.27 1.27)) (justify left bottom))
+  )
   (label "REGN" (at 419.1 207.645 0) (fields_autoplaced)
     (effects (font (size 1.27 1.27)) (justify left bottom))
@@
     (effects (font (size 1.27 1.27)) (justify left bottom))
   )
+  (label "VBUS" (at 299.085 185.42 0) (fields_autoplaced)
+    (effects (font (size 1.27 1.27)) (justify left bottom))
+  )
   (label "GPIO7" (at 162.56 160.02 0) (fields_autoplaced)
     (effects (font (size 1.27 1.27)) (justify left bottom))
@@
   (label "GPIO8" (at 135.255 302.26 180) (fields_autoplaced)
     (effects (font (size 1.27 1.27)) (justify right bottom))
+  )
+  (label "VSYS" (at 219.075 131.445 0) (fields_autoplaced)
+    (effects (font (size 1.27 1.27)) (justify left bottom))
   )
   (label "GPIO10" (at 135.255 294.64 180) (fields_autoplaced)
@@
     )
   )
-  (symbol (lib_id "power:+5V") (at 299.085 185.42 0) (unit 1)
-    (in_bom yes) (on_board yes) (dnp no) (fields_autoplaced)
-    (property "Reference" "#PWR025" (at 299.085 189.23 0)
-      (effects (font (size 1.27 1.27)) hide)
-    )
-    (property "Value" "+5V" (at 299.085 180.975 0)
-      (effects (font (size 1.27 1.27)))
-    )
-    (property "Footprint" "" (at 299.085 185.42 0)
-      (effects (font (size 1.27 1.27)) hide)
-    )
-    (property "Datasheet" "" (at 299.085 185.42 0)
-      (effects (font (size 1.27 1.27)) hide)
-    )
-    (pin "1")
-    (instances
-      (project "carrier_board_v1"
-        (path "/7c2e4356-99de-4c13-89ad-ca928a2db042/fc4c71a5-1008-4ac4-98db-57c838c57d91"
-          (reference "#PWR025") (unit 1)
-        )
-      )
-    )
-  )
   (symbol (lib_name "GND_2") (lib_id "power:GND") (at 511.81 241.935 0) (unit 1)
     (in_bom yes) (on_board yes) (dnp no) (fields_autoplaced)
@@
         )
       )
-    )
-  )
-  (symbol (lib_id "power:+5V") (at 485.14 152.4 270) (unit 1)
-    (in_bom yes) (on_board yes) (dnp no) (fields_autoplaced)
-    (property "Reference" "#PWR014" (at 481.33 152.4 0)
-      (effects (font (size 1.27 1.27)) hide)
-    )
-    (property "Value" "+5V" (at 488.95 152.4 90)
-      (effects (font (size 1.27 1.27)) (justify left))
-    )
-    (property "Footprint" "" (at 485.14 152.4 0)
-      (effects (font (size 1.27 1.27)) hide)
-    )
-    (property "Datasheet" "" (at 485.14 152.4 0)
-      (effects (font (size 1.27 1.27)) hide)
-    )
-    (pin "1")
-    (instances
-      (project "carrier_board_v1"
-        (path "/7c2e4356-99de-4c13-89ad-ca928a2db042/fc4c71a5-1008-4ac4-98db-57c838c57d91"
-          (reference "#PWR014") (unit 1)
-        )
-      )

Commit message: -
Parts:
- removed L3: 1uH, Inductor_SMD:L_0603_1608Metric, symbol dk_Fixed-Inductors:82473C
- removed U2: TPS61256YFFR, YFF0009ACAG, symbol TPS61256YFFR:TPS61256YFFR
- added C7: 10uF, Capacitor_SMD:C_0603_1608Metric, symbol Device:C
- added L1: 13R106C, digikey-footprints:Inductor_13R106C, symbol dk_Fixed-Inductors:13R106C
- added U4: MP28167GQ-P, QFN-16_MP28167GQ_MNP, symbol MP28167GQ-P:MP28167GQ-P
- C1: value 10uF -> 0.1
- C9: value 10uF -> 100
- Module1: footprint CM4IO:Raspberry-Pi-4-Compute-Module -> DF40C-100DS-0.4V_51_:HRS_DF40C-100DS-0.4V(51)
Connections:
- net +5V: no longer C1.1, C8.1
- net GND: now also C7.2
- net PMID: no longer C9.1, U1.15 (PMID)
- net at C6.1, J1.2, L2.2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: no longer Q1.5 (D)
- new net: C1.1, C7.1, C8.1, C9.1, U4.12 (OUT)
Other:
- moved on the sheet: C2, D1, Q1, R5

Commit message: -
Parts:
- removed U4: MP28167GQ-P, QFN-16_MP28167GQ_MNP, symbol MP28167GQ-P:MP28167GQ-P
- added C10: 100nF, Capacitor_SMD:C_0603_1608Metric, symbol Device:C
- added C11: 1uF, Capacitor_SMD:C_0603_1608Metric, symbol Device:C
- added C12, C13: 22nF, Capacitor_SMD:C_0603_1608Metric, symbol Device:C
- added C14: 0.1uF, Capacitor_SMD:C_0603_1608Metric, symbol Device:C
- added C15: 22uF, Capacitor_SMD:C_0603_1608Metric, symbol Device:C
- added C16: 100uF, symbol Device:C_Polarized_US
- added R7: 499kΩ, Resistor_SMD:R_0603_1608Metric, symbol Device:R
- added U2: MP28167GQ-P, QFN-16_MP28167GQ_MNP, symbol MP28167GQ-P:MP28167GQ-P
- C1: value 0.1 -> 100uF
- C8: value 10uF -> 0.1uF
- C9: value 100 -> 100nF
- D1: footprint Diode_SMD:D_SMA -> Diode_SMD:D_0603_1608Metric
- L1: value 13R106C -> 4.7uH; footprint digikey-footprints:Inductor_13R106C -> digikey-footprints:0603
- Module1: footprint DF40C-100DS-0.4V_51_:HRS_DF40C-100DS-0.4V(51) -> CM4IO:Raspberry-Pi-4-Compute-Module
- R5: value 1.1 -> 21.5k
Connections:
- net +5V: now also D1.1 (K), Q1.1 (S), Q1.2 (S), Q1.3 (S)
- net GND: now also C11.1, C12.2, C13.2, C14.2, C15.2, C16.2, U2.10 (AGND), U2.11 (GND), U2.2 (GND), U2.5 (RSV1), U2.6 (RSV2); no longer C9.2
- net PMID: now also U1.15 (PMID); no longer C2.1, Q1.1 (S), Q1.2 (S), Q1.3 (S)
- net at C1.1, C7.1, C8.1: now also C2.1, Q1.5 (D), U2.12 (OUT); no longer C9.1
- net at L1.1: now also C10.1, U2.14 (SW2)
- net at L1.2: now also C9.1, U2.15 (SW1)
- net at C6.1, J1.2, L2.2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: now also C14.1, C15.1, C16.1, R7.2, U2.1 (IN)
- net VBUS: no longer names the net of C3.1, CR1.1, D1.2 (A), J6.A4_B9 (VBUS), J6.B4_A9 (VBUS), U1.16 (VBUS)
- net VBUS: now also Q1.4 (G)
- new net: C13.1, R7.1, U2.3 (EN)
- new net: C10.2, U2.13 (BST2)
- new net: C9.2, U2.16 (BST1)
- new net: C12.1, R5.2, U2.7 (OC)
- new net: C11.2, U2.9 (VCC)
Other:
- moved on the sheet: CR1, J6, R6, R9

Commit message: version 2
Parts:
- removed L2: MAKK2016T1R0M, INDC2016X100N, symbol MAKK2016T1R0M:MAKK2016T1R0M
- added C17: 2.2uF, Capacitor_SMD:C_0603_1608Metric, symbol Device:C
- added L3: 1uH, digikey-footprints:0603, symbol dk_Fixed-Inductors:13R106C
- C16: footprint (none) -> Capacitor_SMD:C_0603_1608Metric
- C5: value 2.2u -> 2.2uF
- J7: footprint Connector_PinHeader_2.54mm:PinHeader_1x12_P2.54mm_Vertical -> Connector_PinSocket_1.27mm:PinSocket_1x12_P1.27mm_Vertical
- U2: footprint QFN-16_MP28167GQ_MNP -> MP28167GQ-P:QFN-16_MP28167GQ_MNP
Connections:
- net GND: now also C17.1
- net at C4.2, U1.13 (SW): now also L3.2
- net at C14.1, C15.1, C16.1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: now also L3.1
- net PMID: no longer names the net of U1.15 (PMID)
- net PMID: now also C17.2
Changed lines of the file:
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@@
     (stroke (width 0) (type default))
   )
-  (wire (pts (xy 413.385 192.405) (xy 414.655 192.405))
+  (wire (pts (xy 413.385 192.405) (xy 417.195 192.405))
     (stroke (width 0) (type default))
   )
@@
     (stroke (width 0) (type default))
   )
+  (wire (pts (xy 345.44 200.025) (xy 342.9 200.025))
+    (stroke (width 0) (type default))
+  )
   (wire (pts (xy 264.16 212.725) (xy 266.065 212.725))
     (stroke (width 0) (type default))
@@
     (stroke (width 0) (type default))
   )
-  (wire (pts (xy 429.895 192.405) (xy 451.485 192.405))
+  (wire (pts (xy 427.355 192.405) (xy 451.485 192.405))
     (stroke (width 0) (type default))
   )
@@
     (stroke (width 0) (type solid))
   )
-  (wire (pts (xy 349.25 200.025) (xy 353.06 200.025))
-    (stroke (width 0) (type default))
-  )
   (wire (pts (xy 400.05 197.485) (xy 393.7 197.485))
     (stroke (width 0) (type default))
@@
   )
   (wire (pts (xy 159.385 220.98) (xy 166.37 220.98))
+    (stroke (width 0) (type default))
+  )
+  (wire (pts (xy 342.9 200.025) (xy 342.9 201.295))
     (stroke (width 0) (type default))
   )
@@
   (label "GPIO2" (at 93.98 185.42 180) (fields_autoplaced)
     (effects (font (size 1.27 1.27)) (justify right bottom))
-  )
-  (label "PMID" (at 349.25 200.025 0) (fields_autoplaced)
-    (effects (font (size 1.27 1.27)) (justify left bottom))
   )
   (label "GPIO11" (at 87.63 160.02 0) (fields_autoplaced)
@@
       (effects (font (size 1.27 1.27)) (justify left))
     )
-    (property "Value" "2.2u" (at 322.58 214.63 0)
+    (property "Value" "2.2uF" (at 322.58 214.63 0)
       (effects (font (size 1.27 1.27)) (justify left))
     )
@@
       (effects (font (size 1.524 1.524)))
     )
-    (property "Footprint" "QFN-16_MP28167GQ_MNP" (at 418.465 104.14 0)
+    (property "Footprint" "MP28167GQ-P:QFN-16_MP28167GQ_MNP" (at 418.465 104.14 0)
       (effects (font (size 1.27 1.27) italic) hide)
     )
@@
     )
   )
-  (symbol (lib_id "MAKK2016T1R0M:MAKK2016T1R0M") (at 422.275 192.405 0) (unit 1)
-    (in_bom yes) (on_board yes) (dnp no) (fields_autoplaced)
-    (property "Reference" "L2" (at 422.275 186.055 0)
-      (effects (font (size 1.27 1.27)))
-    )
-    (property "Value" "MAKK2016T1R0M" (at 422.275 188.595 0)
-      (effects (font (size 1.27 1.27)))
-    )
-    (property "Footprint" "INDC2016X100N" (at 422.275 192.405 0)
-      (effects (font (size 1.27 1.27)) (justify bottom) hide)
-    )
-    (property "Datasheet" "" (at 422.275 192.405 0)
-      (effects (font (size 1.27 1.27)) hide)
-    )
-    (pin "1")
-    (pin "2")
-    (instances
-      (project "carrier_board_v1"
-        (path "/7c2e4356-99de-4c13-89ad-ca928a2db042/fc4c71a5-1008-4ac4-98db-57c838c57d91"
-          (reference "L2") (unit 1)
-        )
-      )
-    )
-  )
   (symbol (lib_name "GND_4") (lib_id "power:GND") (at 362.585 121.92 0) (unit 1)
     (in_bom yes) (on_board yes) (dnp no)
@@
       (effects (font (size 1.27 1.27)) (justify left))
     )
-    (property "Footprint" "" (at 487.68 107.95 0)
+    (property "Footprint" "Capacitor_SMD:C_0603_1608Metric" (at 487.68 107.95 0)
       (effects (font (size 1.27 1.27)) hide)
     )
@@
       (effects (font (size 1.27 1.27)))
     )
-    (property "Footprint" "Connector_PinHeader_2.54mm:PinHeader_1x12_P2.54mm_Vertical" (at 120.015 297.18 0)
+    (property "Footprint" "Connector_PinSocket_1.27mm:PinSocket_1x12_P1.27mm_Vertical" (at 120.015 297.18 0)
       (effects (font (size 1.27 1.27)) hide)
     )
@@
     )
   )
+  (symbol (lib_name "GND_3") (lib_id "power:GND") (at 342.9 201.295 0) (unit 1)
+    (in_bom yes) (on_board yes) (dnp no) (fields_autoplaced)
+    (property "Reference" "#PWR034" (at 342.9 207.645 0)
+      (effects (font (size 1.27 1.27)) hide)
+    )
+    (property "Value" "GND" (at 342.9 206.375 0)
+      (effects (font (size 1.27 1.27)))
+    )
+    (property "Footprint" "" (at 342.9 201.295 0)
+      (effects (font (size 1.27 1.27)) hide)
+    )
+    (property "Datasheet" "" (at 342.9 201.295 0)
+      (effects (font (size 1.27 1.27)) hide)
+    )
+    (pin "1")
+    (instances
+      (project "carrier_board_v1"
+        (path "/7c2e4356-99de-4c13-89ad-ca928a2db042/fc4c71a5-1008-4ac4-98db-57c838c57d91"
+          (reference "#PWR034") (unit 1)
+        )
+      )
+    )
+  )
   (symbol (lib_id "Device:R") (at 411.48 207.645 90) (unit 1)
     (in_bom yes) (on_board yes) (dnp no)
@@
         (path "/7c2e4356-99de-4c13-89ad-ca928a2db042/fc4c71a5-1008-4ac4-98db-57c838c57d91"
           (reference "#PWR030") (unit 1)
+        )
+      )
+    )
+  )
+  (symbol (lib_id "Device:C") (at 349.25 200.025 90) (unit 1)
+    (in_bom yes) (on_board yes) (dnp no)
+    (property "Reference" "C17" (at 353.695 201.295 90)
+      (effects (font (size 1.27 1.27)))
+    )
+    (property "Value" "2.2uF" (at 353.695 203.835 90)
+      (effects (font (size 1.27 1.27)))
+    )
+    (property "Footprint" "Capacitor_SMD:C_0603_1608Metric" (at 353.06 199.0598 0)
+      (effects (font (size 1.27 1.27)) hide)
+    )
+    (property "Datasheet" "~" (at 349.25 200.025 0)
+      (effects (font (size 1.27 1.27)) hide)
+    )
+    (pin "1")
+    (pin "2")
+    (instances
+      (project "carrier_board_v1"
+        (path "/7c2e4356-99de-4c13-89ad-ca928a2db042/fc4c71a5-1008-4ac4-98db-57c838c57d91"
+          (reference "C17") (unit 1)
         )
       )
@@
         )
       )
+    )
+  )
+  (symbol (lib_id "dk_Fixed-Inductors:13R106C") (at 422.275 192.405 180) (unit 1)
+    (in_bom yes) (on_board yes) (dnp no)
+    (property "Reference" "L3" (at 421.64 186.055 0)
+      (effects (font (size 1.524 1.524)) (justify right))
+    )
+    (property "Value" "1uH" (at 421.64 188.595 0)
+      (effects (font (size 1.524 1.524)) (justify right))
+    )
+    (property "Footprint" "digikey-footprints:0603" (at 417.195 197.485 0)
+      (effects (font (size 1.524 1.524)) (justify left) hide)
+    )
+    (property "Datasheet" "https://www.murata-ps.com/data/magnetics/kmp_1300r.pdf" (at 417.195 200.025 0)
+      (effects (font (size 1.524 1.524)) (justify left) hide)
+    )
+    (property "Digi-Key_PN" "811-2058-ND" (at 417.195 202.565 0)
+      (effects (font (size 1.524 1.524)) (justify left) hide)
+    )
+    (property "MPN" "13R106C" (at 417.195 205.105 0)
+      (effects (font (size 1.524 1.524)) (justify left) hide)
+    )
+    (property "Category" "Inductors, Coils, Chokes" (at 417.195 207.645 0)
+      (effects (font (size 1.524 1.524)) (justify left) hide)
+    )
+    (property "Family" "Fixed Inductors" (at 417.195 210.185 0)
+      (effects (font (size 1.524 1.524)) (justify left) hide)
+    )
+    (property "DK_Datasheet_Link" "https://www.murata-ps.com/data/magnetics/kmp_1300r.pdf" (at 417.195 212.725 0)
+      (effects (font (size 1.524 1.524)) (justify left) hide)
+    )
+    (property "DK_Detail_Page" "/product-detail/en/murata-power-solutions-inc/13R106C/811-2058-ND/1998245" (at 417.195 215.265 0)
+      (effects (font (size 1.524 1.524)) (justify left) hide)
+    )
+    (property "Description" "FIXED IND 10MH 85MA 23.8 OHM TH" (at 417.195 217.805 0)
+      (effects (font (size 1.524 1.524)) (justify left) hide)
+    )
+    (property "Manufacturer" "Murata Power Solutions Inc." (at 417.195 220.345 0)
+      (effects (font (size 1.524 1.524)) (justify left) hide)
+    )
+    (property "Status" "Active" (at 417.195 222.885 0)
+      (effects (font (size 1.524 1.524)) (justify left) hide)
+    )
+    (pin "1")
+    (pin "2")
+    (instances
+      (project "carrier_board_v1"
+        (path "/7c2e4356-99de-4c13-89ad-ca928a2db042/fc4c71a5-1008-4ac4-98db-57c838c57d91"
+          (reference "L3") (unit 1)
+        )
+      )

Commit message: almost
Parts:
- removed J7: Conn_01x12_Pin, Connector_PinSocket_1.27mm:PinSocket_1x12_P1.27mm_Vertical, symbol Connector:Conn_01x12_Pin
- added C18, C19, C20: 10uF, Capacitor_SMD:C_0603_1608Metric, symbol Device:C
- added J5: C2938398, Connector_PinSocket_1.27mm:PinSocket_2x08_P1.27mm_Vertical_SMD, symbol Connector:Conn_01x16_Socket
- C1, C16: footprint Capacitor_SMD:C_0603_1608Metric -> Capacitor_Tantalum_SMD:CP_EIA-3528-21_Kemet-B
- J6: value USB4105-GF-A -> C2997432
- L1, L3: footprint digikey-footprints:0603 -> Inductor_SMD:L_0805_2012Metric
- Module1: value ComputeModule4-CM4 -> DF40C-100DS-0.4V(51)
Connections:
- net +3.3V: now also J5.4 (Pin_4), J5.6 (Pin_6)
- net +5V: now also C18.1, C19.1, C20.1
- net GND: now also C18.2, C19.2, C20.2, J5.1 (Pin_1), J5.12 (Pin_12), J5.16 (Pin_16), J5.5 (Pin_5)
- net GPIO10: now also J5.10 (Pin_10)
- net GPIO11: now also J5.11 (Pin_11)
- net GPIO14: now also J5.14 (Pin_14)
- net GPIO15: now also J5.15 (Pin_15)
- net GPIO2: now also J5.2 (Pin_2)
- net GPIO3: now also J5.3 (Pin_3)
- net GPIO7: now also J5.7 (Pin_7)
- net GPIO8: now also J5.8 (Pin_8)
- net GPIO9: now also J5.9 (Pin_9)
- net nRPIBOOT: now also J5.13 (Pin_13)

Commit message: complete
Parts:
- removed L1: 4.7uH, Inductor_SMD:L_0805_2012Metric, symbol dk_Fixed-Inductors:13R106C
- added L2: SRP5030CA-2R2M, SRP5030CA4R7M, symbol SRP5030CA-2R2M:SRP5030CA-2R2M
- C12: value 22nF -> 33nF
- C20: value 10uF -> 100nF
- J1: value B2B-PH-SM4-TB_LF__SN_ -> C157930
- R5: value 21.5k -> 15k
Connections:
- net at C10.1, U2.14 (SW2): now also L2.2
- net at C9.1, U2.15 (SW1): now also L2.1
Other:
- moved on the sheet: C20

Commit message: -
Parts:
- removed D1: CDBA340-HF, Diode_SMD:D_0603_1608Metric, symbol Diode:CDBA340-HF
- added J2: DF40C-100DS-0.4V(51), HRS_DF40C-100DS-0.4V(51), symbol DF40C-100DS-0.4V_51_:DF40C-100DS-0.4V(51)
- added U4: CDBA340-HF, CDBA-HF, symbol CDBA340-HF:CDBA340-HF
Connections:
- net +3.3V: now also J5.13 (Pin_13), J5.14 (Pin_14), J5.15 (Pin_15), J5.16 (Pin_16); no longer J5.4 (Pin_4), J5.6 (Pin_6)
- net +5V: now also U4.1
- net GND: now also J5.10 (Pin_10), J5.11 (Pin_11), J5.8 (Pin_8), J5.9 (Pin_9); no longer J5.16 (Pin_16), J5.5 (Pin_5)
- net at C3.1, CR1.1, J6.A4_B9 (VBUS)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: now also U4.2
- net GPIO6: now reaches Module1.30 (GPIO6)
- net GPIO6: now also J5.6 (Pin_6)
- net GPIO5: now reaches Module1.34 (GPIO5)
- net GPIO5: now also J5.5 (Pin_5)
- net GPIO27: now reaches Module1.48 (GPIO27)
- net GPIO27: now also J5.7 (Pin_7)
- net GPIO4: now reaches Module1.54 (GPIO4)
- net GPIO4: now also J5.4 (Pin_4)
- net GPIO10: no longer names the net of Module1.44 (GPIO10)
- net GPIO10: no longer J5.10 (Pin_10)
- net GPIO11: no longer names the net of Module1.38 (GPIO11)
- net GPIO11: no longer J5.11 (Pin_11)
- net GPIO14: no longer names the net of Module1.55 (GPIO14)
- net GPIO14: no longer J5.14 (Pin_14)
- net GPIO15: no longer names the net of Module1.51 (GPIO15)
- net GPIO15: no longer J5.15 (Pin_15)
- net GPIO7: no longer names the net of Module1.37 (GPIO7)
- net GPIO7: no longer J5.7 (Pin_7)
- net GPIO8: no longer names the net of Module1.39 (GPIO8)
- net GPIO8: no longer J5.8 (Pin_8)
- net GPIO9: no longer names the net of Module1.40 (GPIO9)
- net GPIO9: no longer J5.9 (Pin_9)
- net nRPIBOOT: no longer names the net of Module1.93 (nRPIBOOT)
- net nRPIBOOT: no longer J5.13 (Pin_13)
- no-connect marks 66 -> 70
