File: cm4-high-speed.kicad_sch (KiCad schematic)
At the start: 10 parts, among them J3 54548-2271, J3 USB4105-GF-A, U3 TPD2EUSB30

Commit message: schematic almost ready
Parts:
- removed R5, R6: 2.2K 1%, Resistor_SMD:R_0402_1005Metric, symbol Device:R
Connections:
- net +3.3V: no longer names the net of J3.22
- net SCL1: no longer names the net of J3.20
- net SCL1: no longer J3.21

Commit message: schematic complete
Connections:
- net +3.3v: now also J3.22
- net SCL0: now also J3.20
- net SDA0: now also J3.21
Changed lines of the file:
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@@
     (stroke (width 0) (type solid))
   )
-  (wire (pts (xy 221.615 174.625) (xy 234.95 174.625))
+  (wire (pts (xy 218.44 174.625) (xy 234.95 174.625))
     (stroke (width 0) (type default))
   )
@@
     (stroke (width 0) (type solid))
   )
-  (wire (pts (xy 229.87 186.69) (xy 213.36 186.69))
+  (wire (pts (xy 234.95 184.785) (xy 218.44 184.785))
     (stroke (width 0) (type solid))
   )
@@
     (stroke (width 0) (type default))
   )
-  (wire (pts (xy 229.87 189.23) (xy 213.36 189.23))
+  (wire (pts (xy 234.95 187.325) (xy 218.44 187.325))
     (stroke (width 0) (type solid))
   )
@@
     (stroke (width 0) (type solid))
   )
-  (wire (pts (xy 229.87 184.15) (xy 213.36 184.15))
+  (wire (pts (xy 234.95 182.245) (xy 218.44 182.245))
     (stroke (width 0) (type solid))
   )
@@
     (effects (font (size 1.27 1.27)) (justify right bottom))
   )
-  (label "SDA0" (at 213.36 186.69 0) (fields_autoplaced)
+  (label "SDA0" (at 218.44 184.785 0) (fields_autoplaced)
     (effects (font (size 1.27 1.27)) (justify left bottom))
   )
@@
     (effects (font (size 1.27 1.27)) (justify left bottom))
   )
-  (label "+3.3v" (at 213.36 189.23 0) (fields_autoplaced)
+  (label "+3.3v" (at 218.44 187.325 0) (fields_autoplaced)
     (effects (font (size 1.27 1.27)) (justify left bottom))
   )
@@
     (effects (font (size 1.27 1.27)) (justify left bottom))
   )
-  (label "SCL0" (at 213.36 184.15 0) (fields_autoplaced)
+  (label "SCL0" (at 218.44 182.245 0) (fields_autoplaced)
     (effects (font (size 1.27 1.27)) (justify left bottom))
   )
@@
     (effects (font (size 1.27 1.27)) (justify right bottom))
   )
-  (hierarchical_label "+3.3v" (shape input) (at 213.36 189.23 180) (fields_autoplaced)
+  (global_label "SDA0" (shape input) (at 218.44 184.785 180) (fields_autoplaced)
     (effects (font (size 1.27 1.27)) (justify right))
-  )
-  (hierarchical_label "SDA0" (shape input) (at 213.36 186.69 180) (fields_autoplaced)
+    (property "Intersheetrefs" "${INTERSHEET_REFS}" (at 210.6615 184.785 0)
+      (effects (font (size 1.27 1.27)) (justify right) hide)
+    )
+  )
+  (global_label "CAM_GPIO" (shape input) (at 218.44 174.625 180) (fields_autoplaced)
     (effects (font (size 1.27 1.27)) (justify right))
-  )
-  (hierarchical_label "SCL0" (shape input) (at 213.36 184.15 180) (fields_autoplaced)
+    (property "Intersheetrefs" "${INTERSHEET_REFS}" (at 206.1862 174.625 0)
+      (effects (font (size 1.27 1.27)) (justify right) hide)
+    )
+  )
+  (global_label "SCL0" (shape input) (at 218.44 182.245 180) (fields_autoplaced)
     (effects (font (size 1.27 1.27)) (justify right))
-  )
-  (hierarchical_label "CAM_GPIO" (shape input) (at 221.615 174.625 180) (fields_autoplaced)
+    (property "Intersheetrefs" "${INTERSHEET_REFS}" (at 210.722 182.245 0)
+      (effects (font (size 1.27 1.27)) (justify right) hide)
+    )
+  )
+  (global_label "+3.3v" (shape input) (at 218.44 187.325 180) (fields_autoplaced)
     (effects (font (size 1.27 1.27)) (justify right))
+    (property "Intersheetrefs" "${INTERSHEET_REFS}" (at 209.8753 187.325 0)
+      (effects (font (size 1.27 1.27)) (justify right) hide)
+    )
   )
   (symbol (lib_id "Power_Protection:TPD2EUSB30") (at 141.605 226.06 0) (unit 1)

Commit message: pää hajoo
Parts:
- R1, R4, R7, R8: footprint Resistor_SMD:R_0603_1608Metric_Pad0.98x0.95mm_HandSolder -> Resistor_SMD:R_0201_0603Metric
Changed lines of the file:
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@@
       (effects (font (size 1.27 1.27)) (justify left))
     )
-    (property "Footprint" "Resistor_SMD:R_0603_1608Metric_Pad0.98x0.95mm_HandSolder" (at 281.559 86.106 90)
+    (property "Footprint" "Resistor_SMD:R_0201_0603Metric" (at 281.559 86.106 90)
       (effects (font (size 1.27 1.27)) hide)
     )
@@
       (effects (font (size 1.27 1.27)) (justify left))
     )
-    (property "Footprint" "Resistor_SMD:R_0603_1608Metric_Pad0.98x0.95mm_HandSolder" (at 220.98 72.771 90)
+    (property "Footprint" "Resistor_SMD:R_0201_0603Metric" (at 220.98 72.771 90)
       (effects (font (size 1.27 1.27)) hide)
     )
@@
       (effects (font (size 1.27 1.27)) (justify left))
     )
-    (property "Footprint" "Resistor_SMD:R_0603_1608Metric_Pad0.98x0.95mm_HandSolder" (at 303.149 93.726 90)
+    (property "Footprint" "Resistor_SMD:R_0201_0603Metric" (at 303.149 93.726 90)
       (effects (font (size 1.27 1.27)) hide)
     )
@@
       (effects (font (size 1.27 1.27)) (justify left))
     )
-    (property "Footprint" "Resistor_SMD:R_0603_1608Metric_Pad0.98x0.95mm_HandSolder" (at 303.149 81.026 90)
-      (effects (font (size 1.27 1.27)) hide)
-    )
+    (property "Footprint" "Resistor_SMD:R_0201_0603Metric" (at 303.149 81.026 90)
+      (effects (font (size 1.27 1.27)) hide)
+    )

Commit message: send help
Parts:
- removed R1: 5.1k, Resistor_SMD:R_0201_0603Metric, symbol Device:R
- added R4: 56k, Resistor_SMD:R_0201_0603Metric, symbol Device:R
- R4: value 5.1k -> 56k
Connections:
- net GND: now also Module1.101 (USB_OTG_ID); no longer R4.2
- net USB_OTG_ID: no longer Module1.101 (USB_OTG_ID)
- net at J3.B5 (CC2): now also R4.2; no longer R4.1
- net VBUS: now reaches J3.A4_B9 (VBUS), J3.B4_A9 (VBUS), R7.1
- net VBUS: now also R4.1, R4.1
- net at J3.A5 (CC1): now also R4.2
Other:
- moved on the sheet: R4

Commit message: -
Parts:
- removed R7, R8: 2.2K 1%, Resistor_SMD:R_0201_0603Metric, symbol Device:R
Changed lines of the file:
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@@
   (junction (at 105.41 173.99) (diameter 1.016) (color 0 0 0 0)
   )
-  (junction (at 304.927 87.376) (diameter 1.016) (color 0 0 0 0)
-  )
   (junction (at 171.45 166.37) (diameter 1.016) (color 0 0 0 0)
   )
@@
   )
   (junction (at 171.45 181.61) (diameter 1.016) (color 0 0 0 0)
-  )
-  (junction (at 286.004 74.676) (diameter 0) (color 0 0 0 0)
   )
   (junction (at 224.917 84.836) (diameter 0) (color 0 0 0 0)
@@
     (stroke (width 0) (type solid))
   )
-  (wire (pts (xy 304.927 87.376) (xy 304.927 89.916))
-    (stroke (width 0) (type solid))
-  )
   (wire (pts (xy 168.91 158.75) (xy 171.45 158.75))
     (stroke (width 0) (type solid))
@@
     (stroke (width 0) (type solid))
   )
-  (wire (pts (xy 290.957 87.376) (xy 304.927 87.376))
-    (stroke (width 0) (type solid))
-  )
   (wire (pts (xy 233.045 156.845) (xy 233.045 164.465))
     (stroke (width 0) (type default))
@@
     (stroke (width 0) (type solid))
   )
-  (wire (pts (xy 286.004 74.676) (xy 304.927 74.676))
-    (stroke (width 0) (type default))
-  )
   (wire (pts (xy 222.377 84.836) (xy 224.917 84.836))
     (stroke (width 0) (type default))
@@
     (stroke (width 0) (type solid))
   )
-  (wire (pts (xy 304.927 84.836) (xy 304.927 87.376))
-    (stroke (width 0) (type solid))
-  )
   (wire (pts (xy 105.41 120.65) (xy 105.41 128.27))
     (stroke (width 0) (type solid))
@@
     (stroke (width 0) (type solid))
   )
-  (wire (pts (xy 304.927 74.676) (xy 304.927 77.216))
-    (stroke (width 0) (type solid))
-  )
   (wire (pts (xy 286.004 74.676) (xy 286.004 79.756))
     (stroke (width 0) (type default))
@@
   (wire (pts (xy 233.045 179.705) (xy 233.045 197.485))
     (stroke (width 0) (type default))
-  )
-  (wire (pts (xy 304.927 97.536) (xy 304.927 100.076))
-    (stroke (width 0) (type solid))
   )
   (wire (pts (xy 233.045 172.085) (xy 234.95 172.085))
@@
   )
   (label "CAM0_C_P" (at 219.71 154.305 0) (fields_autoplaced)
-    (effects (font (size 1.27 1.27)) (justify left bottom))
-  )
-  (label "USB_OTG_ID" (at 290.957 87.376 0) (fields_autoplaced)
     (effects (font (size 1.27 1.27)) (justify left bottom))
   )
@@
     )
   )
-  (symbol (lib_id "power:GND") (at 304.927 100.076 0) (unit 1)
-    (in_bom yes) (on_board yes) (dnp no)
-    (property "Reference" "#PWR014" (at 304.927 106.426 0)
-      (effects (font (size 1.27 1.27)) hide)
-    )
-    (property "Value" "GND" (at 306.197 105.156 0)
-      (effects (font (size 1.27 1.27)))
-    )
-    (property "Footprint" "" (at 304.927 100.076 0)
-      (effects (font (size 1.27 1.27)) hide)
-    )
-    (property "Datasheet" "" (at 304.927 100.076 0)
-      (effects (font (size 1.27 1.27)) hide)
-    )
-    (pin "1")
-    (instances
-      (project "carrier_board_v1"
-        (path "/7c2e4356-99de-4c13-89ad-ca928a2db042/caa71f4c-454d-4ac9-b287-456eafb34991"
-          (reference "#PWR014") (unit 1)
-        )
-      )
-      (project "rpi-cm4-base-carrier"
-        (path "/9fe8d829-2397-4498-9aed-cc1af0780e59/caa71f4c-454d-4ac9-b287-456eafb34991"
-          (reference "#PWR0115") (unit 1)
-        )
-      )
-    )
-  )
   (symbol (lib_id "power:GND") (at 141.605 238.76 0) (unit 1)
     (in_bom yes) (on_board yes) (dnp no)
@@
         (path "/9fe8d829-2397-4498-9aed-cc1af0780e59/caa71f4c-454d-4ac9-b287-456eafb34991"
           (reference "#PWR0113") (unit 1)
-        )
-      )
-    )
-  )
-  (symbol (lib_id "Device:R") (at 304.927 93.726 0) (unit 1)
-    (in_bom yes) (on_board yes) (dnp no)
-    (property "Reference" "R8" (at 307.467 92.456 0)
-      (effects (font (size 1.27 1.27)) (justify left))
-    )
-    (property "Value" "2.2K 1%" (at 307.467 93.726 0)
-      (effects (font (size 1.27 1.27)) (justify left))
-    )
-    (property "Footprint" "Resistor_SMD:R_0201_0603Metric" (at 303.149 93.726 90)
-      (effects (font (size 1.27 1.27)) hide)
-    )
-    (property "Datasheet" "~" (at 304.927 93.726 0)
-      (effects (font (size 1.27 1.27)) hide)
-    )
-    (property "Manufacturer" "Yageo" (at 304.927 93.726 0)
-      (effects (font (size 1.27 1.27)) hide)
-    )
-    (property "MPN" "RC0603FR-072K2L" (at 304.927 93.726 0)
-      (effects (font (size 1.27 1.27)) hide)
-    )
-    (property "Digi-Key_PN" "311-2.20KHRCT-ND" (at 304.927 93.726 0)
-      (effects (font (size 1.27 1.27)) hide)
-    )
-    (pin "1")
-    (pin "2")
-    (instances
-      (project "carrier_board_v1"
-        (path "/7c2e4356-99de-4c13-89ad-ca928a2db042/caa71f4c-454d-4ac9-b287-456eafb34991"
-          (reference "R8") (unit 1)
-        )
-      )
-      (project "rpi-cm4-base-carrier"
-        (path "/9fe8d829-2397-4498-9aed-cc1af0780e59/caa71f4c-454d-4ac9-b287-456eafb34991"
-          (reference "R8") (unit 1)
         )
       )
@@
         )
       )
-    )
-  )
-  (symbol (lib_id "Device:R") (at 304.927 81.026 0) (unit 1)
-    (in_bom yes) (on_board yes) (dnp no)
-    (property "Reference" "R7" (at 307.467 79.756 0)
-      (effects (font (size 1.27 1.27)) (justify left))
-    )
-    (property "Value" "2.2K 1%" (at 307.467 81.026 0)
-      (effects (font (size 1.27 1.27)) (justify left))
-    )
-    (property "Footprint" "Resistor_SMD:R_0201_0603Metric" (at 303.149 81.026 90)
-      (effects (font (size 1.27 1.27)) hide)
-    )
-    (property "Datasheet" "~" (at 304.927 81.026 0)
-      (effects (font (size 1.27 1.27)) hide)
-    )
-    (property "Manufacturer" "Yageo" (at 304.927 81.026 0)
-      (effects (font (size 1.27 1.27)) hide)
-    )
-    (property "MPN" "RC0603FR-072K2L" (at 304.927 81.026 0)
-      (effects (font (size 1.27 1.27)) hide)
-    )
-    (property "Digi-Key_PN" "311-2.20KHRCT-ND" (at 304.927 81.026 0)
-      (effects (font (size 1.27 1.27)) hide)
-    )
-    (pin "1")
-    (pin "2")
-    (instances
-      (project "carrier_board_v1"
-        (path "/7c2e4356-99de-4c13-89ad-ca928a2db042/caa71f4c-454d-4ac9-b287-456eafb34991"
-          (reference "R7") (unit 1)
-        )
-      )
-      (project "rpi-cm4-base-carrier"
-        (path "/9fe8d829-2397-4498-9aed-cc1af0780e59/caa71f4c-454d-4ac9-b287-456eafb34991"
-          (reference "R7") (unit 1)
-        )
-      )

Commit message: what the fuck
Connections:
- net VBUS renamed +5V
Changed lines of the file:
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@@
     (stroke (width 0) (type solid))
   )
-  (wire (pts (xy 282.575 70.485) (xy 282.575 74.676))
+  (wire (pts (xy 282.575 70.612) (xy 282.575 74.676))
     (stroke (width 0) (type default))
   )
@@
     (effects (font (size 1.27 1.27)) (justify left bottom))
   )
-  (label "VBUS" (at 282.575 70.485 0) (fields_autoplaced)
-    (effects (font (size 1.27 1.27)) (justify left bottom))
-  )
   (label "CAM0_D1_N" (at 219.71 144.145 0) (fields_autoplaced)
     (effects (font (size 1.27 1.27)) (justify left bottom))
@@
     (effects (font (size 1.27 1.27)) (justify left bottom))
   )
-  (label "VBUS" (at 219.202 67.31 0) (fields_autoplaced)
-    (effects (font (size 1.27 1.27)) (justify left bottom))
-  )
   (label "USB2_P" (at 212.852 82.296 180) (fields_autoplaced)
     (effects (font (size 1.27 1.27)) (justify right bottom))
@@
     )
   )
+  (global_label "+5V" (shape input) (at 282.575 70.612 90)
+    (effects (font (size 1.27 1.27)) (justify left))
+    (property "Intersheetrefs" "${INTERSHEET_REFS}" (at 282.575 70.612 0)
+      (effects (font (size 1.27 1.27)) hide)
+    )
+  )
+  (global_label "+5V" (shape input) (at 219.202 67.31 90)
+    (effects (font (size 1.27 1.27)) (justify left))
+    (property "Intersheetrefs" "${INTERSHEET_REFS}" (at 219.202 67.31 0)
+      (effects (font (size 1.27 1.27)) hide)
+    )
+  )
   (global_label "+3.3v" (shape input) (at 218.44 187.325 180) (fields_autoplaced)
     (effects (font (size 1.27 1.27)) (justify right))
@@
     )
   )
+  (netclass_flag "" (length 2.54) (shape round) (at 261.493 102.616 0) (fields_autoplaced)
+    (effects (font (size 1.27 1.27)) (justify left bottom))
+    (property "Netclass" "USB Data" (at 262.382 100.076 0)
+      (effects (font (size 1.27 1.27) italic) (justify left) hide)
+    )
+  )
+  (netclass_flag "" (length 2.54) (shape round) (at 216.916 82.296 0) (fields_autoplaced)
+    (effects (font (size 1.27 1.27)) (justify left bottom))
+    (property "Netclass" "USB Data" (at 217.805 79.756 0)
+      (effects (font (size 1.27 1.27) italic) (justify left) hide)
+    )
+  )

Commit message: -
Connections:
- net +3.3v renamed +3.3V
- no-connect marks 59 -> 69
Changed lines of the file:
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@@
   (no_connect (at 168.91 184.15))
   (no_connect (at 168.91 176.53))
-  (no_connect (at 168.275 161.29))
+  (no_connect (at 168.91 161.29))
   (no_connect (at 107.95 148.59))
   (no_connect (at 227.457 87.376))
   (no_connect (at 168.91 130.81))
+  (no_connect (at 168.91 87.63))
   (no_connect (at 107.95 140.97))
   (no_connect (at 107.95 179.07))
   (no_connect (at 168.91 179.07))
   (no_connect (at 107.95 168.91))
+  (no_connect (at 168.91 110.49))
   (no_connect (at 107.95 85.09))
   (no_connect (at 168.91 163.83))
@@
   (no_connect (at 168.91 123.19))
   (no_connect (at 107.95 123.19))
+  (no_connect (at 168.91 80.01))
+  (no_connect (at 168.91 100.33))
   (no_connect (at 107.95 130.81))
   (no_connect (at 168.91 138.43))
@@
   (no_connect (at 234.95 192.405))
   (no_connect (at 107.95 163.83))
+  (no_connect (at 168.91 107.95))
   (no_connect (at 107.95 77.47))
   (no_connect (at 234.95 167.005))
@@
   (no_connect (at 168.91 153.67))
   (no_connect (at 107.95 153.67))
+  (no_connect (at 168.91 85.09))
+  (no_connect (at 168.91 102.87))
   (no_connect (at 107.95 125.73))
+  (no_connect (at 168.91 77.47))
   (no_connect (at 168.91 120.65))
   (no_connect (at 107.95 133.35))
+  (no_connect (at 168.91 92.71))
   (no_connect (at 168.91 118.11))
   (no_connect (at 168.91 156.21))
@@
   (no_connect (at 107.95 146.05))
   (no_connect (at 107.95 115.57))
+  (no_connect (at 168.91 95.25))
   (no_connect (at 168.91 113.03))
   (no_connect (at 268.097 87.376))
@@
     (stroke (width 0) (type solid))
   )
+  (wire (pts (xy 91.44 92.71) (xy 107.95 92.71))
+    (stroke (width 0) (type default))
+  )
   (wire (pts (xy 141.605 236.22) (xy 141.605 238.76))
     (stroke (width 0) (type solid))
@@
     (stroke (width 0) (type solid))
   )
-  (wire (pts (xy 107.95 92.71) (xy 91.44 92.71))
-    (stroke (width 0) (type solid))
+  (wire (pts (xy 218.44 187.325) (xy 234.95 187.325))
+    (stroke (width 0) (type default))
   )
   (wire (pts (xy 268.097 84.836) (xy 275.082 84.836))
@@
     (stroke (width 0) (type default))
   )
-  (wire (pts (xy 107.95 102.87) (xy 91.44 102.87))
+  (wire (pts (xy 91.44 102.87) (xy 107.95 102.87))
     (stroke (width 0) (type solid))
   )
@@
     (stroke (width 0) (type default))
   )
+  (wire (pts (xy 91.44 100.33) (xy 107.95 100.33))
+    (stroke (width 0) (type default))
+  )
   (wire (pts (xy 171.45 173.99) (xy 171.45 181.61))
     (stroke (width 0) (type solid))
@@
     (stroke (width 0) (type default))
   )
-  (wire (pts (xy 107.95 95.25) (xy 91.44 95.25))
-    (stroke (width 0) (type solid))
-  )
   (wire (pts (xy 214.757 82.296) (xy 227.457 82.296))
     (stroke (width 0) (type default))
@@
     (stroke (width 0) (type solid))
   )
-  (wire (pts (xy 107.95 100.33) (xy 91.44 100.33))
-    (stroke (width 0) (type solid))
-  )
   (wire (pts (xy 222.377 84.836) (xy 224.917 84.836))
     (stroke (width 0) (type default))
@@
     (stroke (width 0) (type solid))
   )
+  (wire (pts (xy 91.44 95.25) (xy 107.95 95.25))
+    (stroke (width 0) (type default))
+  )
   (wire (pts (xy 168.91 181.61) (xy 171.45 181.61))
     (stroke (width 0) (type solid))
@@
     (stroke (width 0) (type default))
   )
-  (wire (pts (xy 234.95 187.325) (xy 218.44 187.325))
-    (stroke (width 0) (type solid))
-  )
   (wire (pts (xy 168.91 74.93) (xy 171.45 74.93))
     (stroke (width 0) (type solid))
@@
     (effects (font (size 1.27 1.27)) (justify left bottom))
   )
-  (label "CAM0_D0_N" (at 102.87 92.71 180) (fields_autoplaced)
+  (label "CAM0_D0_N" (at 91.44 92.71 180) (fields_autoplaced)
     (effects (font (size 1.27 1.27)) (justify right bottom))
   )
@@
     (effects (font (size 1.27 1.27)) (justify left bottom))
   )
-  (label "CAM0_D1_N" (at 102.87 100.33 180) (fields_autoplaced)
-    (effects (font (size 1.27 1.27)) (justify right bottom))
-  )
-  (label "CAM0_D1_P" (at 102.87 102.87 180) (fields_autoplaced)
+  (label "CAM0_D1_N" (at 91.44 100.33 180) (fields_autoplaced)
+    (effects (font (size 1.27 1.27)) (justify right bottom))
+  )
+  (label "CAM0_D1_P" (at 91.44 102.87 180) (fields_autoplaced)
     (effects (font (size 1.27 1.27)) (justify right bottom))
   )
@@
     (effects (font (size 1.27 1.27)) (justify left bottom))
   )
-  (label "+3.3v" (at 218.44 187.325 0) (fields_autoplaced)
+  (label "+3.3V" (at 218.44 187.325 0) (fields_autoplaced)
     (effects (font (size 1.27 1.27)) (justify left bottom))
   )
@@
     (effects (font (size 1.27 1.27)) (justify right bottom))
   )
-  (label "CAM0_D0_P" (at 102.87 95.25 180) (fields_autoplaced)
+  (label "CAM0_D0_P" (at 91.44 95.25 180) (fields_autoplaced)
     (effects (font (size 1.27 1.27)) (justify right bottom))
   )
@@
     )
   )
-  (global_label "+3.3v" (shape input) (at 218.44 187.325 180) (fields_autoplaced)
+  (global_label "+3.3V" (shape input) (at 218.44 187.325 180) (fields_autoplaced)
     (effects (font (size 1.27 1.27)) (justify right))
-    (property "Intersheetrefs" "${INTERSHEET_REFS}" (at 209.8753 187.325 0)
+    (property "Intersheetrefs" "${INTERSHEET_REFS}" (at 209.7543 187.325 0)
       (effects (font (size 1.27 1.27)) (justify right) hide)
     )
@@
       (effects (font (size 1.27 1.27) italic) (justify left) hide)
     )
+  )
+  (netclass_flag "" (length 2.54) (shape round) (at 273.431 79.756 0) (fields_autoplaced)
+    (effects (font (size 1.27 1.27)) (justify left bottom))
+    (property "Netclass" "Power" (at 274.32 77.216 0)
+      (effects (font (size 1.27 1.27) italic) (justify left) hide)
+    )
+  )
+  (netclass_flag "" (length 2.54) (shape round) (at 223.266 79.756 0) (fields_autoplaced)
+    (effects (font (size 1.27 1.27)) (justify left bottom))
+    (property "Netclass" "Power" (at 224.155 77.216 0)
+      (effects (font (size 1.27 1.27) italic) (justify left) hide)
+    )

Commit message: -
Parts:
- R4: value 56k -> 56kΩ; footprint Resistor_SMD:R_0201_0603Metric -> Resistor_SMD:R_0402_1005Metric
Changed lines of the file:
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@@
       (effects (font (size 1.27 1.27)) (justify left))
     )
-    (property "Value" "56k" (at 280.289 82.042 90)
+    (property "Value" "56kΩ" (at 280.289 82.042 90)
       (effects (font (size 1.27 1.27)) (justify left))
     )
-    (property "Footprint" "Resistor_SMD:R_0201_0603Metric" (at 282.194 77.978 90)
+    (property "Footprint" "Resistor_SMD:R_0402_1005Metric" (at 282.194 77.978 90)
       (effects (font (size 1.27 1.27)) hide)
     )
@@
       (effects (font (size 1.27 1.27)) (justify left))
     )
-    (property "Value" "56k" (at 220.472 72.517 0)
+    (property "Value" "56kΩ" (at 220.472 72.517 0)
       (effects (font (size 1.27 1.27)) (justify left))
     )
-    (property "Footprint" "Resistor_SMD:R_0201_0603Metric" (at 217.424 72.771 90)
-      (effects (font (size 1.27 1.27)) hide)
-    )
+    (property "Footprint" "Resistor_SMD:R_0402_1005Metric" (at 217.424 72.771 90)
+      (effects (font (size 1.27 1.27)) hide)
+    )
