File: cm4-high-speed.kicad_sch (KiCad schematic)
At the start: 6 parts, among them J3 54548-2271, J3 USB4105-GF-A, U3 TPD2EUSB30

Commit message: final commit
Parts:
- R4: footprint Resistor_SMD:R_0402_1005Metric -> Resistor_SMD:R_0603_1608Metric
Changed lines of the file:
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@@
       (effects (font (size 1.27 1.27)) (justify left))
     )
-    (property "Footprint" "Resistor_SMD:R_0402_1005Metric" (at 282.194 77.978 90)
+    (property "Footprint" "Resistor_SMD:R_0603_1608Metric" (at 282.194 77.978 90)
       (effects (font (size 1.27 1.27)) hide)
     )
@@
       (effects (font (size 1.27 1.27)) (justify left))
     )
-    (property "Footprint" "Resistor_SMD:R_0402_1005Metric" (at 217.424 72.771 90)
-      (effects (font (size 1.27 1.27)) hide)
-    )
+    (property "Footprint" "Resistor_SMD:R_0603_1608Metric" (at 217.424 72.771 90)
+      (effects (font (size 1.27 1.27)) hide)
+    )

Commit message: -
Parts:
- Module1: footprint CM4IO:Raspberry-Pi-4-Compute-Module -> DF40C-100DS-0.4V_51_:HRS_DF40C-100DS-0.4V(51); Field4 Hirose -> (none); Field5 2x DF40C-100DS-0.4V -> (none); MPN (Alt) 2x DF40HC(3.0)-100DS-0.4V -> (none)
Changed lines of the file:
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@@
       (effects (font (size 1.27 1.27)))
     )
-    (property "Footprint" "CM4IO:Raspberry-Pi-4-Compute-Module" (at 140.97 147.32 0)
+    (property "Footprint" "DF40C-100DS-0.4V_51_:HRS_DF40C-100DS-0.4V(51)" (at 140.97 147.32 0)
       (effects (font (size 1.27 1.27)) hide)
     )
     (property "Datasheet" "" (at 140.97 147.32 0)
-      (effects (font (size 1.27 1.27)) hide)
-    )
-    (property "Field4" "Hirose" (at 138.43 52.07 0)
-      (effects (font (size 1.27 1.27)) hide)
-    )
-    (property "Field5" "2x DF40C-100DS-0.4V" (at 138.43 54.61 0)
       (effects (font (size 1.27 1.27)) hide)
     )
@@
       (effects (font (size 1.27 1.27)) hide)
     )
-    (property "MPN (Alt)" "2x DF40HC(3.0)-100DS-0.4V" (at 102.87 31.115 0)
-      (effects (font (size 1.27 1.27)) hide)
-    )

Commit message: -
Parts:
- Module1: footprint DF40C-100DS-0.4V_51_:HRS_DF40C-100DS-0.4V(51) -> CM4IO:Raspberry-Pi-4-Compute-Module; Field4 (none) -> Hirose; Field5 (none) -> 2x DF40C-100DS-0.4V; MPN (Alt) (none) -> 2x DF40HC(3.0)-100DS-0.4V
Changed lines of the file:
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@@
       (effects (font (size 1.27 1.27)))
     )
-    (property "Footprint" "DF40C-100DS-0.4V_51_:HRS_DF40C-100DS-0.4V(51)" (at 140.97 147.32 0)
+    (property "Footprint" "CM4IO:Raspberry-Pi-4-Compute-Module" (at 140.97 147.32 0)
       (effects (font (size 1.27 1.27)) hide)
     )
     (property "Datasheet" "" (at 140.97 147.32 0)
+      (effects (font (size 1.27 1.27)) hide)
+    )
+    (property "Field4" "Hirose" (at 138.43 52.07 0)
+      (effects (font (size 1.27 1.27)) hide)
+    )
+    (property "Field5" "2x DF40C-100DS-0.4V" (at 138.43 54.61 0)
       (effects (font (size 1.27 1.27)) hide)
     )
@@
       (effects (font (size 1.27 1.27)) hide)
     )
+    (property "MPN (Alt)" "2x DF40HC(3.0)-100DS-0.4V" (at 102.87 31.115 0)
+      (effects (font (size 1.27 1.27)) hide)
+    )

Commit message: almost
Parts:
- J3: value USB4105-GF-A -> C2997432
- J3: value 54548-2271 -> C262390
- Module1: value ComputeModule4-CM4 -> DF40C-100DS-0.4V(51); Field4 Hirose -> (none); Field5 2x DF40C-100DS-0.4V -> (none); MPN (Alt) 2x DF40HC(3.0)-100DS-0.4V -> (none)
- U3: value TPD2EUSB30 -> TPD2EUSB30DRTR
Connections:
- net GND: now also J3.SH1 (SHIELD), J3.SH2 (SHIELD)
- no-connect marks 69 -> 68
Changed lines of the file:
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@@
   (junction (at 105.41 158.75) (diameter 1.016) (color 0 0 0 0)
+  )
+  (junction (at 233.045 192.405) (diameter 0) (color 0 0 0 0)
   )
   (junction (at 105.41 128.27) (diameter 1.016) (color 0 0 0 0)
@@
   (no_connect (at 107.95 161.29))
   (no_connect (at 107.95 80.01))
-  (no_connect (at 234.95 192.405))
   (no_connect (at 107.95 163.83))
   (no_connect (at 168.91 107.95))
@@
     (stroke (width 0) (type solid))
   )
+  (wire (pts (xy 233.045 192.405) (xy 233.045 197.485))
+    (stroke (width 0) (type default))
+  )
   (wire (pts (xy 219.202 76.581) (xy 219.202 79.756))
     (stroke (width 0) (type default))
@@
     (stroke (width 0) (type solid))
   )
+  (wire (pts (xy 233.045 192.405) (xy 234.95 192.405))
+    (stroke (width 0) (type default))
+  )
   (wire (pts (xy 171.45 90.17) (xy 171.45 97.79))
     (stroke (width 0) (type solid))
@@
     (stroke (width 0) (type solid))
   )
-  (wire (pts (xy 233.045 179.705) (xy 233.045 197.485))
+  (wire (pts (xy 233.045 179.705) (xy 233.045 192.405))
     (stroke (width 0) (type default))
   )
@@
       (effects (font (size 1.27 1.27)))
     )
-    (property "Value" "TPD2EUSB30" (at 141.605 218.44 0)
+    (property "Value" "TPD2EUSB30DRTR" (at 141.605 218.44 0)
       (effects (font (size 1.27 1.27)))
     )
@@
       (effects (font (size 1.27 1.27)))
     )
-    (property "Value" "USB4105-GF-A" (at 248.9494 69.6624 0)
+    (property "Value" "C2997432" (at 248.9494 69.6624 0)
       (effects (font (size 1.27 1.27)))
     )
@@
       (effects (font (size 1.27 1.27)) hide)
     )
-    (property "Value" "ComputeModule4-CM4" (at 139.065 53.975 0)
+    (property "Value" " DF40C-100DS-0.4V(51)" (at 139.065 53.975 0)
       (effects (font (size 1.27 1.27)))
     )
@@
       (effects (font (size 1.27 1.27)) hide)
     )
-    (property "Field4" "Hirose" (at 138.43 52.07 0)
-      (effects (font (size 1.27 1.27)) hide)
-    )
-    (property "Field5" "2x DF40C-100DS-0.4V" (at 138.43 54.61 0)
-      (effects (font (size 1.27 1.27)) hide)
-    )
     (property "Digi-Key_PN" "2x H11615CT-ND" (at -1.27 120.65 0)
       (effects (font (size 1.27 1.27)) hide)
@@
     )
     (property "MPN" "2x DF40C-100DS-0.4V" (at 102.87 33.655 0)
-      (effects (font (size 1.27 1.27)) hide)
-    )
-    (property "MPN (Alt)" "2x DF40HC(3.0)-100DS-0.4V" (at 102.87 31.115 0)
       (effects (font (size 1.27 1.27)) hide)
     )
@@
       (effects (font (size 1.27 1.27)) (justify left))
     )
-    (property "Value" "54548-2271" (at 252.73 156.21 0)
+    (property "Value" "C262390" (at 252.73 156.21 0)
       (effects (font (size 1.27 1.27)) (justify left))
     )

Commit message: -
Parts:
- removed J3: C262390, 54548-2271:MOLEX_54548-2271, symbol 54548-2271:54548-2271
- added J3: FH34SRJ-22S-0.5SH50, CONN22x1_FH34SRJ-22S-0.5SH50_HIR, symbol FH34SRJ-22S-0-5SH-50:FH34SRJ-22S-0.5SH50
- added J7: DF40C-100DS-0.4V(51), HRS_DF40C-100DS-0.4V(51), symbol DF40C-100DS-0.4V_51_:DF40C-100DS-0.4V(51)
- R4: value 56kΩ -> 5.1k
Connections:
- net +3.3V: now also J3.22
- net +5V: no longer R4.1, R4.1
- net CAM0_C_N: now also J3.8
- net CAM0_C_P: now also J3.9
- net CAM0_D0_N: now also J3.2
- net CAM0_D0_P: now also J3.3
- net CAM0_D1_N: now also J3.5
- net CAM0_D1_P: now also J3.6
- net CAM_GPIO: now also J3.17
- net GND: now also R4.1, R4.1, J3.1, J3.10, J3.13, J3.16, J3.18, J3.19, J3.4, J3.7
- net SCL0: now also J3.20
- net SDA0: now also J3.21
- no-connect marks 68 -> 67

Commit message: -
Connections:
- net GND: now also J3.S1 (SHELL_GND), J3.S2 (SHELL_GND), J3.S3 (SHELL_GND), J3.S4 (SHELL_GND)
Changed lines of the file:
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@@
   (junction (at 214.757 82.296) (diameter 0) (color 0 0 0 0)
+  )
+  (junction (at 270.637 94.996) (diameter 0) (color 0 0 0 0)
   )
   (junction (at 235.585 174.625) (diameter 0) (color 0 0 0 0)
@@
     (stroke (width 0) (type solid))
   )
+  (wire (pts (xy 268.097 94.996) (xy 270.637 94.996))
+    (stroke (width 0) (type default))
+  )
   (wire (pts (xy 282.575 70.612) (xy 282.575 74.676))
     (stroke (width 0) (type default))
@@
   (wire (pts (xy 168.91 181.61) (xy 171.45 181.61))
     (stroke (width 0) (type solid))
+  )
+  (wire (pts (xy 270.637 96.9772) (xy 270.637 94.996))
+    (stroke (width 0) (type default))
   )
   (wire (pts (xy 105.41 151.13) (xy 105.41 158.75))
@@
     )
   )
-  (symbol (lib_id "power:GND") (at 270.637 94.996 0) (unit 1)
+  (symbol (lib_id "power:GND") (at 270.637 96.9772 0) (unit 1)
     (in_bom yes) (on_board yes) (dnp no)
-    (property "Reference" "#PWR04" (at 270.637 101.346 0)
-      (effects (font (size 1.27 1.27)) hide)
-    )
-    (property "Value" "GND" (at 271.907 100.076 0)
+    (property "Reference" "#PWR04" (at 270.637 103.3272 0)
+      (effects (font (size 1.27 1.27)) hide)
+    )
+    (property "Value" "GND" (at 270.6116 100.6348 0)
       (effects (font (size 1.27 1.27)))
     )
-    (property "Footprint" "" (at 270.637 94.996 0)
-      (effects (font (size 1.27 1.27)) hide)
-    )
-    (property "Datasheet" "" (at 270.637 94.996 0)
-      (effects (font (size 1.27 1.27)) hide)
-    )
+    (property "Footprint" "" (at 270.637 96.9772 0)
+      (effects (font (size 1.27 1.27)) hide)
+    )
+    (property "Datasheet" "" (at 270.637 96.9772 0)
+      (effects (font (size 1.27 1.27)) hide)
+    )

Commit message: version3 complete
Parts:
- J7: footprint HRS_DF40C-100DS-0.4V(51) -> DF40C-100DS-0.4V_51_:HRS_DF40C-100DS-0.4V(51)
Changed lines of the file:
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@@
       (effects (font (size 1.27 1.27)))
     )
-    (property "Footprint" "HRS_DF40C-100DS-0.4V(51)" (at 41.91 160.02 0)
+    (property "Footprint" "DF40C-100DS-0.4V_51_:HRS_DF40C-100DS-0.4V(51)" (at 41.91 160.02 0)
       (effects (font (size 1.27 1.27)) (justify bottom) hide)
     )
