File: _autosave-cm4-gpio.kicad_sch (KiCad schematic)
At the start: 25 parts, among them J1 B2B-PH-SM4-TB_LF__SN_, J6 USB4105-GF-A, J7 Conn_01x12_Pin, Q1 DMP3013SFV, U1 BQ25302RTER, U2 TPS61256YFFR

Commit message: -
Connections:
- net PMID: now also U2.B3 (EN)
Changed lines of the file:
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@@
   (junction (at 248.285 131.445) (diameter 0) (color 0 0 0 0)
+  )
+  (junction (at 314.96 123.825) (diameter 0) (color 0 0 0 0)
   )
   (junction (at 159.385 210.82) (diameter 0) (color 0 0 0 0)
@@
     (stroke (width 0) (type default))
   )
+  (wire (pts (xy 302.26 146.685) (xy 314.96 146.685))
+    (stroke (width 0) (type default))
+  )
   (wire (pts (xy 231.775 197.485) (xy 231.775 198.755))
     (stroke (width 0) (type default))
@@
     (stroke (width 0) (type default))
   )
+  (wire (pts (xy 314.96 123.825) (xy 327.025 123.825))
+    (stroke (width 0) (type default))
+  )
   (wire (pts (xy 158.115 160.02) (xy 162.56 160.02))
     (stroke (width 0) (type default))
@@
     (stroke (width 0) (type default))
   )
+  (wire (pts (xy 314.96 146.685) (xy 314.96 123.825))
+    (stroke (width 0) (type default))
+  )
   (wire (pts (xy 318.77 207.645) (xy 353.06 207.645))
     (stroke (width 0) (type default))
@@
     (stroke (width 0) (type default))
   )
-  (wire (pts (xy 306.705 123.825) (xy 327.025 123.825))
-    (stroke (width 0) (type default))
-  )
+  (wire (pts (xy 306.705 123.825) (xy 314.96 123.825))
+    (stroke (width 0) (type default))
+  )
